File: SBC.kicad_pcb (KiCad board)
At the start: 2 copper layers, 160 x 100.3 mm, 93 parts, among them K1 CONN_3, K10 CONN_3, K11 CONN_3, K12 CONN_3, K13 CONN_3, K2 CONN_3, K3 CONN_3, K4 CONN_3, K5 CONN_3, K6 CONN_3, K7 CONN_3, K8 CONN_3, K9 CONN_3, P1 PARALLEL, P2 POWER, P3 SERIAL, P4 CLK_CPU, P5 CLK_UART, P6 RESET, SW1 SW_PUSH, U1 16550, U10 74LS243, U11 74LS245, U12 74LS174, U13 74LS174, U14 74LS32, U15 74LS32, U16 74LS32, U17 74LS244, U18 74LS174, U19 8255, U2 27C080, U20 C96ABC, U21 DS1302, U22 MAX232, U23 SRAM_512KO, U24 Z80-CPU, U25 DS1210, U26 74LS06N, U3 74LS08, U4 74LS10, U5 74LS125, U6 74LS139, U7 74LS14, U8 74LS245, U9 74LS245, X1 CRYSTAL

Commit message: Version B
Parts:
- added LS1: Speaker, Connector_PinHeader_2.54mm:PinHeader_2x01_P2.54mm_Vertical, F.Cu at (113.7, 56.0)
- added Q1: 2N3906, Package_TO_SOT_THT:TO-92_Inline, F.Cu at (118.0, 56.6)
- added R13: 3K6, Resistor_THT:R_Axial_DIN0204_L3.6mm_D1.6mm_P7.62mm_Horizontal, F.Cu at (117.9, 81.4)
- added R14: 3K6, Resistor_THT:R_Axial_DIN0204_L3.6mm_D1.6mm_P7.62mm_Horizontal, F.Cu at (116.5, 68.6)
- added R15: 120R, Resistor_THT:R_Axial_DIN0204_L3.6mm_D1.6mm_P7.62mm_Horizontal, F.Cu at (113.7, 61.0)
- BT1, JP1, JP2, P6: footprint SIL-2 -> Connector_PinHeader_2.54mm:PinHeader_1x02_P2.54mm_Vertical
- C1, C10, C11, C12, C13, C14, C15, C16, C17, C18, C19, C20, C21, C22, C23, C29, C3, C30, C32, C4, C5, C6, C7, C8, C9: footprint C2 -> Capacitor_THT:C_Disc_D7.0mm_W2.5mm_P5.00mm
- C2, C31: footprint C1V5 -> Capacitor_THT:CP_Radial_D5.0mm_P2.50mm
- C24, C25, C26, C27, C28: footprint C1V5 -> Capacitor_THT:CP_Radial_Tantal_D4.5mm_P2.50mm
- D1: footprint LEDV -> LED_THT:LED_D5.0mm
- D2: value DIODE -> 1N4148; footprint D3 -> Diode_THT:D_DO-35_SOD27_P7.62mm_Horizontal
- K1, K10, K11, K12, K13, K2, K3, K4, K5, K6, K7, K8, K9: footprint SIL-3 -> Connector_PinHeader_2.54mm:PinHeader_1x03_P2.54mm_Vertical
- P1: footprint pin_array_13x2 -> Connector_PinHeader_2.54mm:PinHeader_2x13_P2.54mm_Vertical
- P3: footprint PIN_ARRAY_5x2 -> Connector_PinHeader_2.54mm:PinHeader_2x05_P2.54mm_Vertical
- P4: footprint 8dip300 -> Package_DIP:DIP-8_W7.62mm_Socket
- P5: footprint 8dip300 -> Oscillator:Oscillator_DIP-8
- R1: value 10 -> 10R; footprint R3 -> Resistor_THT:R_Axial_DIN0204_L3.6mm_D1.6mm_P7.62mm_Horizontal
- R11, R12, R2, R9: footprint R3 -> Resistor_THT:R_Axial_DIN0204_L3.6mm_D1.6mm_P7.62mm_Horizontal
- RR1, RR2: footprint SIL-6 -> Resistor_THT:R_Array_SIP6
- SW1: footprint SW_PUSH_SMALL -> Button_Switch_THT:SW_PUSH_6mm_H8mm
- U1, U19, U24: footprint 40dip600 -> Package_DIP:DIP-40_W15.24mm
- U10, U14, U15, U16, U26, U3, U4, U5, U7: footprint 14dip300 -> Package_DIP:DIP-14_W7.62mm
- U11, U17, U8, U9: footprint 20dip300 -> Package_DIP:DIP-20_W7.62mm
- U12, U13, U18, U22, U6: footprint 16dip300 -> Package_DIP:DIP-16_W7.62mm
- U2, U23: footprint 32dip600 -> Package_DIP:DIP-32_W15.24mm
- U21, U25: footprint 8dip300 -> Package_DIP:DIP-8_W7.62mm
- X1: footprint SIL-2 -> Crystal:Crystal_Round_D3.0mm_Vertical
- moved U1 25.3 mm to (125.7, 91.4), turned to 90 degrees
- moved U19 25.3 mm to (125.7, 71.1), turned to 90 degrees
- moved U24 25.3 mm to (125.7, 151.1), turned to 90 degrees
- moved U2 20.5 mm to (125.7, 130.8), turned to 90 degrees
- moved U23 20.5 mm to (125.7, 111.8), turned to 90 degrees
- moved P1 15.3 mm to (82.5, 86.4), turned to 180 degrees
- moved U11 12.0 mm to (195.6, 63.5), turned to 90 degrees
- moved U17 12.0 mm to (195.6, 141.0), turned to 90 degrees
- moved U8 12.0 mm to (195.6, 74.9), turned to 90 degrees
- moved U9 12.0 mm to (195.6, 151.1), turned to 90 degrees
- moved U12 9.67 mm to (96.5, 120.7), turned to 90 degrees
- moved U13 9.67 mm to (96.5, 130.8), turned to 90 degrees
- moved U18 9.67 mm to (96.5, 90.2), turned to 90 degrees
- moved U6 9.67 mm to (96.5, 141.0), turned to 90 degrees
- moved U22 9.67 mm to (96.5, 110.5), turned to 90 degrees
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Connections:
- D2 pad 1: Net-(C2-Pad1) -> VCC
- D2 pad 2: VCC -> Net-(C2-Pad1)
Routing:
- net GND: track 833.8 -> 881.5 mm, vias 1 -> 2
- net VCC: track 788.3 -> 829.7 mm
- net Net-(Q1-Pad2): track 0.00 -> 27.5 mm
- net Net-(R13-Pad2): track 0.00 -> 20.5 mm
- net Net-(Q1-Pad3): track 0.00 -> 18.4 mm
- net Net-(Q1-Pad1): track 0.00 -> 13.1 mm
- net /PB7: track 90.6 -> 102.3 mm
- net /PC6: track 74.7 -> 85.7 mm
- net //HALT: track 69.6 -> 58.9 mm
- net Net-(U23-Pad22): track 42.0 -> 52.7 mm
- net Net-(C24-Pad1): track 22.0 -> 14.7 mm
- net //RD: track 274.0 -> 281.2 mm
- net //BUSAK: track 136.3 -> 143.5 mm
- net /A10: track 127.4 -> 134.4 mm
- net /D4: track 307.0 -> 313.6 mm
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Other:
- board text added: "19-Jan-2019 Phillip Summers difficultylevelhigh@gmail.com"

Commit message: Version C
Parts:
- JP1: value JUMPER -> BATSEL
- JP2: value JUMPER -> 1BIT-INPUT
- LS1: value Speaker -> SPEAKER
- R12, RR2: value 4700 -> 4K7
- R14: value 3K6 -> 1K8
- R9: value 100 -> 100R
- RR1: value 1000 -> 1K
- SW1: value SW_PUSH -> RESETSW
- moved Q1 2.54 mm to (120.5, 56.6), turned to 180 degrees
Connections:
- Q1 pad 1: Net-(Q1-Pad1) -> VCC
- R14 pad 1: Net-(Q1-Pad1) -> Net-(R14-Pad1)
Routing:
- net Net-(Q1-Pad1): track 13.1 -> 0.00 mm
- net Net-(Q1-Pad3): track 18.4 -> 23.8 mm
- net VCC: track 829.7 -> 834.3 mm
- net Net-(C2-Pad1): track 61.7 -> 64.2 mm

Commit message: Version D
Parts:
- C10, C11, C12, C13, C14, C15, C16, C17, C18, C19, C20, C21, C22, C29, C3, C30, C32, C4, C5, C6, C7, C8, C9: value 0.1 uF -> 0.1uF
- C2: value 10 uF -> 10uF
- C24, C25, C26, C27, C28: value 1.0 uF -> 1uF
- C31: value 22 uF -> 22uF
- JP2: value 1BIT-INPUT -> 1BIT-IN
- K1: value CONN_3 -> A17
- K10: value CONN_3 -> BNKSEL
- K11: value CONN_3 -> 16K/32K
- K12: value CONN_3 -> INTSEL
- K13: value CONN_3 -> RSTSEL
- K2, K4: value CONN_3 -> CTS-DSR
- K3, K5: value CONN_3 -> RTS-DTR
- K6: value CONN_3 -> A18
- K7: value CONN_3 -> 128/512
- K8: value CONN_3 -> A19
- K9: value CONN_3 -> PWR
Connections:
- R14 pad 1: Net-(R14-Pad1) -> Net-(Q1-Pad2)
- U1 pad 29: (no net) -> Net-(U1-Pad29)
Routing:
- net Net-(Q1-Pad3): track 23.8 -> 13.8 mm
- net Net-(Q1-Pad2): track 27.5 -> 35.5 mm
- net /RTC_DQ: track 30.1 -> 28.6 mm
- net /RESET: track 116.4 -> 115.6 mm
- net //CS_RTC: track 151.6 -> 151.4 mm, vias 3 -> 2

Commit message: Version E
Parts:
- added JP3: RAMVCC, Jumper:SolderJumper-2_P1.3mm_Open_RoundedPad1.0x1.5mm, B.Cu at (184.2, 92.7)
- added JP4: RAMCS, Jumper:SolderJumper-2_P1.3mm_Open_RoundedPad1.0x1.5mm, B.Cu at (188.1, 92.7)
- C1, C23: value 0.1 uF -> 0.1uF
- moved D1 25.3 mm to (81.0, 148.5), turned to 0 degrees
- moved R9 20.6 mm to (87.8, 133.6), turned to 90 degrees
- moved P2 10.2 mm to (81.3, 132.1)
- moved BT1 2.54 mm to (80.0, 113.0), turned to 0 degrees
Routing:
- net Net-(D1-Pad1): track 70.3 -> 95.6 mm
- net Net-(K10-Pad2): track 153.4 -> 145.5 mm
- net //IOSEL: track 219.0 -> 211.2 mm
- net GND: track 881.5 -> 887.5 mm
- net VCC: track 834.3 -> 829.9 mm
- net Net-(U16-Pad1): track 231.8 -> 227.4 mm
- net /VCC_SRAM: track 61.9 -> 65.9 mm
- net Net-(JP4-Pad2): track 52.7 -> 48.7 mm
- net /A4: track 153.6 -> 156.4 mm
- net /RTS_TTL: track 51.9 -> 49.2 mm
- net //CS_RAM: track 42.2 -> 44.5 mm
- net /B_/HALT: track 195.9 -> 193.5 mm
- net /A14: track 175.3 -> 173.6 mm
- net /DSR: track 128.1 -> 129.8 mm
- net Net-(K11-Pad2): track 37.7 -> 39.0 mm
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Other:
- board text added: "Beta 21-Jan-2019 Phillip Summers difficultylevelhigh@gmail.com"
- board text removed: "19-Jan-2019 Phillip Summers difficultylevelhigh@gmail.com"

Commit message: Version F
Parts:
- added JP5: TXRX, Connector_PinHeader_2.54mm:PinHeader_1x02_P2.54mm_Vertical, F.Cu at (117.5, 105.8)
- P5: footprint Oscillator:Oscillator_DIP-8 -> Package_DIP:DIP-8_W7.62mm_Socket
- turned P5 to 90 degrees
Routing:
- net VCC: track 829.9 -> 849.7 mm
- net Net-(K10-Pad2): track 145.5 -> 133.8 mm
- net /PC6: track 85.7 -> 75.9 mm
- net /SOUT_TTL: track 48.1 -> 56.3 mm
- net /SIN_TTL: track 44.7 -> 49.1 mm
- net /A0: track 121.0 -> 124.6 mm
- net /PB5: track 94.7 -> 92.8 mm
- net Net-(JP2-Pad2): track 76.7 -> 75.1 mm
- net /VBAT1: track 134.7 -> 133.3 mm
- net Net-(K3-Pad2): track 102.4 -> 103.7 mm
- net /A16_RAM: track 51.5 -> 50.3 mm
- net /PB6: track 91.0 -> 92.2 mm
- net /D7: track 283.4 -> 282.4 mm
- net //CS_CFG: track 26.8 -> 26.0 mm
- net //RTC_WR: track 100.4 -> 101.2 mm
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Other:
- board text added: "Beta 22-Jan-2019 Phillip Summers difficultylevelhigh@gmail.com"
- board text removed: "Beta 21-Jan-2019 Phillip Summers difficultylevelhigh@gmail.com"

Commit message: Version G
Parts:
- removed hole1, hole2: CONN_1, 1pin
- added C33: 0.1uF, Capacitor_THT:C_Disc_D7.0mm_W2.5mm_P5.00mm, F.Cu at (111.0, 61.0)
- added D3: LED, LED_THT:LED_D5.0mm, F.Cu at (87.6, 149.2)
- added R16: 470R, Resistor_THT:R_Axial_DIN0204_L3.6mm_D1.6mm_P7.62mm_Horizontal, F.Cu at (81.0, 144.8)
- added U27: 74LS14, Package_DIP:DIP-14_W7.62mm, F.Cu at (86.5, 60.8)
- P1: value PARALLEL -> IDE; footprint Connector_PinHeader_2.54mm:PinHeader_2x13_P2.54mm_Vertical -> Connector_PinHeader_2.54mm:PinHeader_2x20_P2.54mm_Vertical
- moved K9 31.9 mm to (88.4, 83.7), turned to 0 degrees
- moved P1 30.6 mm to (80.0, 55.9), turned to 0 degrees
- moved C6 25.9 mm to (119.8, 72.4)
- moved P3 13.3 mm to (82.5, 118.7)
- moved C32 8.89 mm to (100.3, 56.0), turned to 0 degrees
- moved BT1 7.84 mm to (87.0, 109.5)
- moved JP2 3.56 mm to (87.1, 118.5)
- moved C9 0.76 mm to (92.2, 83.8)
- moved D1 0.70 mm to (81.0, 149.2)
- moved P2 0.38 mm to (81.3, 132.5)
Connections:
- K9 pad 2: /PPWR -> Net-(K9-Pad2)
- P1 pad 1: /PC0 -> /-PC7
- P1 pad 10: /PA4 -> /PB3
- P1 pad 11: /PC5 -> /PA3
- P1 pad 12: /PA5 -> /PB4
- P1 pad 13: /PC6 -> /PA2
- P1 pad 14: /PA6 -> /PB5
- P1 pad 15: /PC7 -> /PA1
- P1 pad 16: /PA7 -> /PB6
- P1 pad 17: /PB7 -> /PA0
- P1 pad 18: /PB0 -> /PB7
- P1 pad 19: /PB6 -> GND
- P1 pad 2: /PA0 -> GND
- P1 pad 20: /PB1 -> Net-(K9-Pad2)
- P1 pad 21: /PB5 -> Net-(P1-Pad21)
- P1 pad 22: /PB2 -> GND
- P1 pad 23: /PB4 -> /-PC5
- P1 pad 24: /PB3 -> GND
- P1 pad 25: /PPWR -> /-PC6
- P1 pad 3: /PC1 -> /PA7
- P1 pad 4: /PA1 -> /PB0
- P1 pad 5: /PC2 -> /PA6
- P1 pad 6: /PA2 -> /PB1
- P1 pad 7: /PC3 -> /PA5
- P1 pad 8: /PA3 -> /PB2
- P1 pad 9: /PC4 -> /PA4
Routing:
- net /-PC3: track 0.00 -> 45.3 mm, vias 0 -> 1
- net Net-(P1-Pad39): track 0.00 -> 42.3 mm
- net GND: track 887.0 -> 926.8 mm
- net /-PC6: track 0.00 -> 36.4 mm
- net /-PC4: track 0.00 -> 34.7 mm
- net /PC2: track 87.0 -> 112.6 mm
- net /-PC5: track 0.00 -> 24.2 mm
- net /PPWR: track 23.9 -> 0.00 mm
- net /DTR: track 116.1 -> 138.1 mm
- net /DSR: track 129.8 -> 151.7 mm
- net Net-(K9-Pad2): track 0.00 -> 21.3 mm
- net /PB5: track 92.8 -> 112.5 mm, vias 1 -> 2
- net /CTS: track 139.6 -> 158.6 mm
- net /RTS: track 137.0 -> 155.5 mm
- net /PB7: track 102.3 -> 119.2 mm
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Other:
- board text added: "Beta 23-Jan-2019 Phillip Summers difficultylevelhigh@gmail.com"
- board text removed: "Beta 22-Jan-2019 Phillip Summers difficultylevelhigh@gmail.com"

Commit message: Version H
Routing:
- net VCC: track 852.8 -> 873.0 mm
- net /D0: track 269.8 -> 272.7 mm
- net /CTS: track 158.6 -> 157.8 mm
- net /-PC3: track 45.3 -> 44.5 mm
- net Net-(K10-Pad2): track 122.9 -> 122.3 mm

Commit message: Version I
Parts:
- removed D3: LED, LED_THT:LED_D5.0mm
- removed R16: 470R, Resistor_THT:R_Axial_DIN0204_L3.6mm_D1.6mm_P7.62mm_Horizontal
- P1: footprint Connector_PinHeader_2.54mm:PinHeader_2x20_P2.54mm_Vertical -> Connector_IDC:IDC-Header_2x20_P2.54mm_Vertical
- P3: footprint Connector_PinHeader_2.54mm:PinHeader_2x05_P2.54mm_Vertical -> Connector_IDC:IDC-Header_2x05_P2.54mm_Vertical
- P5: footprint Package_DIP:DIP-8_W7.62mm_Socket -> Oscillator:Oscillator_DIP-8
- U27: footprint Package_DIP:DIP-14_W7.62mm -> Package_DIP:DIP-14_W7.62mm_Socket
- moved P2 10.9 mm to (81.3, 143.4)
- moved P3 8.98 mm to (83.2, 127.6)
- moved D1 8.76 mm to (89.8, 149.2)
- moved P1 2.62 mm to (80.6, 58.4)
- moved JP2 1.59 mm to (88.5, 119.3)
- moved BT1 1.52 mm to (88.5, 109.5)
- moved C22 0.51 mm to (91.9, 134.6)
- moved C29 0.51 mm to (91.9, 104.1)
- moved C3 0.51 mm to (91.9, 114.3)
- moved C4 0.51 mm to (91.9, 124.5)
- turned P5 to 0 degrees
Connections:
- P4 pad 2: Net-(P4-Pad2) -> (no net)
- P4 pad 3: Net-(P4-Pad3) -> (no net)
- P4 pad 6: Net-(P4-Pad6) -> (no net)
- P4 pad 7: Net-(P4-Pad7) -> (no net)
Routing:
- net Net-(P1-Pad39): track 42.3 -> 0.00 mm
- net VCC: track 873.0 -> 894.2 mm
- net /TX: track 59.1 -> 77.3 mm
- net /RX: track 51.1 -> 63.2 mm
- net /PA7: track 71.6 -> 60.6 mm
- net /DSR: track 151.7 -> 160.6 mm
- net /DTR: track 138.1 -> 146.6 mm
- net /CTS: track 157.8 -> 165.8 mm
- net /RTS: track 155.5 -> 162.3 mm
- net Net-(D1-Pad1): track 94.4 -> 101.1 mm
- net Net-(D3-Pad2): track 4.95 -> 0.00 mm
- net /-PC4: track 34.7 -> 39.2 mm
- net /PA2: track 54.1 -> 58.4 mm
- net /PC0: track 100.7 -> 104.2 mm
- net //IOSEL: track 207.2 -> 210.6 mm
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