File: SBC.kicad_pcb (KiCad board)
At the start: 2 copper layers, 160 x 100.3 mm, 101 parts, among them K1 A17, K10 BNKSEL, K11 16K/32K, K12 INTSEL, K13 RSTSEL, K2 CTS-DSR, K3 RTS-DTR, K4 CTS-DSR, K5 RTS-DTR, K6 A18, K7 128/512, K8 A19, K9 PWR, P1 IDE, P2 POWER, P3 SERIAL, P4 CLK_CPU, P5 CLK_UART, P6 RESET, Q1 2N3906, SW1 RESETSW, U1 16550, U10 74LS243, U11 74LS245, U12 74LS174, U13 74LS174, U14 74LS32, U15 74LS32, U16 74LS32, U17 74LS244, U18 74LS174, U19 8255, U2 27C080, U20 C96ABC, U21 DS1302, U22 MAX232, U23 SRAM_512KO, U24 Z80-CPU, U25 DS1210, U26 74LS06N, U27 74LS14, U3 74LS08, U4 74LS10, U5 74LS125, U6 74LS139, U7 74LS14, U8 74LS245, U9 74LS245, X1 CRYSTAL

Commit message: Version J
Parts:
- P2: footprint molex-drive-connector -> Connector_BarrelJack:BarrelJack_CUI_PJ-063AH_Horizontal
- U27: footprint Package_DIP:DIP-14_W7.62mm_Socket -> Package_DIP:DIP-14_W7.62mm
- moved Q1 99.3 mm to (87.8, 150.3), turned to 0 degrees
- moved LS1 93.7 mm to (94.9, 147.8), turned to 270 degrees
- moved R15 77.6 mm to (92.9, 135.7)
- moved C18 56.5 mm to (177.2, 61.1)
- moved R13 27.7 mm to (91.6, 72.4)
- moved C22 25.5 mm to (117.5, 135.1)
- moved C33 22.9 mm to (88.4, 64.7), turned to 90 degrees
- moved R14 21.9 mm to (94.9, 72.4), turned to 270 degrees
- moved U27 20.4 mm to (106.8, 59.7), turned to 270 degrees
- moved P5 14.2 mm to (113.0, 65.9)
- moved P2 9.41 mm to (89.9, 139.5), turned to 270 degrees
- moved D1 9.02 mm to (80.8, 149.1)
- moved C32 6.88 mm to (107.2, 56.5), turned to 180 degrees
- moved R9 1.71 mm to (88.6, 132.1)
- moved P6 1.61 mm to (182.6, 56.5), turned to 90 degrees
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Connections:
- P2 pad 1: Net-(P2-Pad1) -> VCC
- U27 pad 1: /PC7 -> /PC4
- U27 pad 2: /-PC7 -> /-PC4
- U27 pad 8: /-PC4 -> /-PC7
- U27 pad 9: /PC4 -> /PC7
Routing:
- net Net-(Q1-Pad2): track 38.5 -> 107.5 mm
- net //IOSEL: track 210.6 -> 243.7 mm
- net /-PC4: track 39.2 -> 63.1 mm
- net /PA4: track 55.9 -> 78.1 mm
- net /-PC3: track 47.1 -> 69.0 mm, vias 1 -> 0
- net Net-(U16-Pad1): track 226.2 -> 244.4 mm
- net /PC3: track 97.3 -> 79.5 mm
- net GND: track 924.7 -> 908.3 mm
- net /CLK_UART: track 83.3 -> 69.6 mm
- net /PC6: track 67.8 -> 54.9 mm
- net /-PC7: track 11.6 -> 24.2 mm
- net /PC7: track 70.7 -> 62.7 mm, vias 1 -> 0
- net Net-(LS1-Pad1): track 4.95 -> 12.9 mm
- net /-PC6: track 33.5 -> 40.8 mm
- net /PB1: track 100.3 -> 94.1 mm
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Other:
- board text added: "Beta 24-Jan-2019 Phillip Summers difficultylevelhigh@gmail.com"
- board text removed: "Beta 23-Jan-2019 Phillip Summers difficultylevelhigh@gmail.com"

Commit message: Version K
Parts:
- D1: value LED -> RUN/HALT
- LS1: value SPEAKER -> SPKR
- P2: footprint Connector_BarrelJack:BarrelJack_CUI_PJ-063AH_Horizontal -> Connector_BarrelJack:BarrelJack_Horizontal
- Q1: footprint Package_TO_SOT_THT:TO-92_Inline -> Package_TO_SOT_THT:TO-92_HandSolder
- moved U27 17.0 mm to (91.6, 67.3), turned to 90 degrees
- moved LS1 14.6 mm to (80.6, 144.8), turned to 0 degrees
- moved R15 8.46 mm to (94.4, 144.0)
- moved Q1 2.61 mm to (90.2, 151.1), turned to 90 degrees
- moved P2 1.94 mm to (91.1, 138.0), turned to 0 degrees
- moved D1 0.83 mm to (80.7, 149.9)
- moved C16 0.63 mm to (121.3, 106.7)
- moved JP5 0.32 mm to (117.8, 105.8)
Connections:
- U27 pad 1: /PC4 -> /PC3
- U27 pad 10: /-PC5 -> Net-(U27-Pad10)
- U27 pad 11: /PC5 -> Net-(U27-Pad11)
- U27 pad 2: /-PC4 -> /-PC3
- U27 pad 3: Net-(U27-Pad3) -> /PC5
- U27 pad 4: Net-(U27-Pad4) -> /-PC5
- U27 pad 5: /PC3 -> /PC4
- U27 pad 6: /-PC3 -> /-PC4
Routing:
- net /PA4: track 78.1 -> 57.6 mm
- net /PC6: track 54.9 -> 69.8 mm, vias 0 -> 1
- net GND: track 908.3 -> 920.6 mm
- net /PC3: track 79.5 -> 91.7 mm
- net /PC7: track 62.7 -> 51.8 mm, vias 0 -> 1
- net /-PC4: track 63.1 -> 53.5 mm
- net /-PC3: track 69.0 -> 60.8 mm
- net /PB5: track 110.2 -> 103.1 mm
- net /-PC7: track 24.2 -> 30.6 mm
- net //IOSEL: track 243.7 -> 238.1 mm
- net /PA2: track 55.3 -> 50.3 mm
- net Net-(C2-Pad1): track 67.5 -> 64.4 mm
- net /PC5: track 60.0 -> 63.0 mm
- net Net-(Q1-Pad3): track 8.06 -> 5.45 mm
- net Net-(Q1-Pad2): track 107.5 -> 105.2 mm
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Other:
- board text added: "Beta 26-Jan-2019 Phillip Summers difficultylevelhigh@gmail.com"
- board text removed: "Beta 24-Jan-2019 Phillip Summers difficultylevelhigh@gmail.com"

Commit message: Version L
Parts:
- U20: footprint C96ABCMC -> library:C96ABCMC
- moved C31 56.0 mm to (227.9, 59.0), turned to 90 degrees
Routing:
- net GND: track 920.6 -> 927.9 mm
- net VCC: track 899.3 -> 900.9 mm

Commit message: Version M
Parts:
- added C4: SUPER, library:SuperCap5, F.Cu at (185.9, 73.0)
Changed lines of the file:
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@@
     (thickness 1.6002)
     (drawings 21)
-    (tracks 4429)
+    (tracks 4428)
     (zones 0)
-    (modules 101)
+    (modules 102)
     (nets 289)
   )
@@
     (36 B.SilkS user)
     (37 F.SilkS user)
-    (38 B.Mask user hide)
-    (39 F.Mask user hide)
+    (38 B.Mask user)
+    (39 F.Mask user)
     (40 Dwgs.User user)
     (41 Cmts.User user)
@@
     (solder_mask_min_width 0.25)
     (aux_axis_origin 0 0)
-    (visible_elements 7FFDFFFF)
+    (visible_elements 7FFFFFFF)
     (pcbplotparams
       (layerselection 0x00030_ffffffff)
@@
     )
   )
+  (module library:SuperCap5 (layer Component)
+    (at 185.8645 73.025)
+    (descr "Condensateur polarise")
+    (tags CP)
+    (fp_text reference C4 (at 1.27 2.54) (layer F.SilkS)
+      (effects (font (size 1.524 1.524) (thickness 0.3048)))
+    )
+    (fp_text value SUPER (at 0 -2.54) (layer F.SilkS)
+      (effects (font (size 1.524 1.3335) (thickness 0.3048)))
+    )
+    (fp_line (start -4.064 0) (end -3.81 0) (layer F.SilkS) (width 0.381))
+    (fp_line (start -4.826 -1.016) (end -4.826 1.016) (layer F.SilkS) (width 0.381))
+    (fp_line (start -4.064 0) (end -5.842 0) (layer F.SilkS) (width 0.381))
+    (fp_circle (center 0 -0.127) (end 6.858 0.127) (layer F.SilkS) (width 0.381))
+    (pad 1 thru_hole rect (at -2.54 0) (size 1.905 1.905) (drill 1.143) (layers *.Cu *.Mask F.SilkS))
+    (pad 2 thru_hole circle (at 2.54 0) (size 1.905 1.905) (drill 1.143) (layers *.Cu *.Mask F.SilkS))
+    (model discret/c_pol.wrl
+      (at (xyz 0 0 0))
+      (scale (xyz 0.5 0.5 0.5))
+      (rotate (xyz 0 0 0))
+    )
+  )
   (gr_text "Beta 26-Jan-2019 Phillip Summers difficultylevelhigh@gmail.com" (at 236.1184 114.7826 90) (layer F.SilkS)
     (effects (font (size 1.016 0.712) (thickness 0.178)))
@@
   (segment (start 86.715633 87.884) (end 86.715633 95.439372) (width 0.2032) (layer Component) (net 114))
   (segment (start 87.11571 87.483923) (end 86.715633 87.884) (width 0.2032) (layer Component) (net 114))
-  (segment (start 180.786675 85.0392) (end 180.3654 85.0392) (width 0.2032) (layer Component) (net 115) (status 30))
-  (segment (start 180.761275 85.1408) (end 180.3654 85.1408) (width 0.2032) (layer Component) (net 115) (status 30))
-  (segment (start 185.95969 83.82) (end 182.082075 83.82) (width 0.2032) (layer Component) (net 115))
-  (segment (start 162.51682 81.50098) (end 163.461724 80.556076) (width 0.2032) (layer Component) (net 115))
+  (segment (start 185.95969 83.82) (end 182.005875 83.82) (width 0.2032) (layer Component) (net 115))
+  (segment (start 186.676401 83.103289) (end 185.95969 83.82) (width 0.2032) (layer Component) (net 115))
+  (segment (start 180.786675 85.0392) (end 180.3654 85.0392) (width 0.2032) (layer Component) (net 115))
   (segment (start 186.676401 81.520401) (end 186.676401 83.103289) (width 0.2032) (layer Component) (net 115))
-  (segment (start 163.461724 80.556076) (end 185.712076 80.556076) (width 0.2032) (layer Component) (net 115))
+  (segment (start 182.005875 83.82) (end 180.786675 85.0392) (width 0.2032) (layer Component) (net 115))
+  (segment (start 185.712076 80.556076) (end 186.676401 81.520401) (width 0.2032) (layer Component) (net 115))
+  (segment (start 143.51 76.2) (end 146.608747 79.298747) (width 0.2032) (layer Component) (net 115))
+  (segment (start 155.323487 79.298747) (end 157.52572 81.50098) (width 0.2032) (layer Component) (net 115))
   (segment (start 157.52572 81.50098) (end 162.51682 81.50098) (width 0.2032) (layer Component) (net 115))
+  (segment (start 162.51682 81.50098) (end 163.461724 80.556076) (width 0.2032) (layer Component) (net 115))
   (segment (start 146.608747 79.298747) (end 155.323487 79.298747) (width 0.2032) (layer Component) (net 115))
-  (segment (start 155.323487 79.298747) (end 157.52572 81.50098) (width 0.2032) (layer Component) (net 115))
-  (segment (start 143.51 76.2) (end 146.608747 79.298747) (width 0.2032) (layer Component) (net 115) (status 10))
-  (segment (start 185.712076 80.556076) (end 186.676401 81.520401) (width 0.2032) (layer Component) (net 115))
-  (segment (start 182.082075 83.82) (end 180.761275 85.1408) (width 0.2032) (layer Component) (net 115) (status 20))
-  (segment (start 186.676401 83.103289) (end 185.95969 83.82) (width 0.2032) (layer Component) (net 115))
+  (segment (start 163.461724 80.556076) (end 185.712076 80.556076) (width 0.2032) (layer Component) (net 115))
   (via (at 160.88106 79.74838) (size 0.889) (layers Component Copper) (net 116))
   (segment (start 175.76292 137.92708) (end 182.88 130.81) (width 0.2032) (layer Copper) (net 116) (status 20))

Commit message: Version N
Parts:
- removed JP5: TXRX, Connector_PinHeader_2.54mm:PinHeader_1x02_P2.54mm_Vertical
- removed K2, K4: CTS-DSR, Connector_PinHeader_2.54mm:PinHeader_1x03_P2.54mm_Vertical
- removed K3, K5: RTS-DTR, Connector_PinHeader_2.54mm:PinHeader_1x03_P2.54mm_Vertical
- added R16: 470R, Resistor_THT:R_Axial_DIN0204_L3.6mm_D1.6mm_P7.62mm_Horizontal, F.Cu at (117.0, 102.9)
- moved D2 11.5 mm to (177.2, 68.5), turned to 270 degrees
- moved C2 9.14 mm to (177.5, 85.9)
- moved C4 7.45 mm to (187.3, 80.3)
- moved C1 1.84 mm to (191.8, 67.3)
- moved C10 1.27 mm to (191.8, 57.1)
Connections:
- P3 pad 2: /DSR -> Net-(P3-Pad2)
- U22 pad 11: Net-(K3-Pad2) -> /RTS_TTL
- U22 pad 12: Net-(K2-Pad2) -> /CTS_TTL
- U22 pad 13: Net-(K4-Pad2) -> /CTS
- U22 pad 14: Net-(K5-Pad2) -> /RTS
Routing:
- net /DSR: track 160.3 -> 0.00 mm, vias 1 -> 0
- net /CTS: track 165.5 -> 46.3 mm, vias 0 -> 1
- net /RTS: track 162.4 -> 45.2 mm, vias 0 -> 1
- net Net-(K4-Pad2): track 113.7 -> 0.00 mm, vias 2 -> 0
- net Net-(K3-Pad2): track 105.0 -> 0.00 mm, vias 1 -> 0
- net Net-(K5-Pad2): track 104.7 -> 0.00 mm, vias 3 -> 0
- net Net-(K2-Pad2): track 95.7 -> 0.00 mm, vias 2 -> 0
- net /DTR: track 146.2 -> 60.3 mm, vias 1 -> 0
- net /RTS_TTL: track 48.5 -> 125.3 mm, vias 0 -> 1
- net /DTR_TTL: track 54.8 -> 0.00 mm
- net /DSR_TTL: track 50.3 -> 0.00 mm
- net /CTS_TTL: track 54.0 -> 103.2 mm, vias 0 -> 2
- net //RESET_IN: track 135.2 -> 122.0 mm
- net GND: track 927.9 -> 937.0 mm
- net /SOUT_TTL: track 57.0 -> 48.1 mm
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
Commit message: Version O
Parts:
- BT1: value BATTERY -> SUPER
- turned C34 to 90 degrees
- renumbered C4 to C34
Connections:
- C34 pad 1: (no net) -> /VBAT1
- C34 pad 2: (no net) -> GND
Routing:
- net /VBAT1: track 124.0 -> 146.8 mm
- net GND: track 937.0 -> 944.0 mm
- net Net-(JP4-Pad2): track 48.3 -> 51.2 mm
- net //CS_RAM: track 44.5 -> 42.8 mm
- net Net-(K11-Pad2): track 38.7 -> 39.9 mm
- net //M1: track 141.8 -> 142.5 mm
- net /A14: track 173.6 -> 174.2 mm

Commit message: Version P
Parts:
- removed BT1: SUPER, Connector_PinHeader_2.54mm:PinHeader_1x02_P2.54mm_Vertical
- C34: value SUPER -> 0.22F
Routing:
- net /VBAT1: track 146.8 -> 114.8 mm
- net GND: track 944.0 -> 943.9 mm, vias 2 -> 3
Other:
- board text added: "Beta 17-Feb-2019 Phillip Summers difficultylevelhigh@gmail.com"
- board text removed: "Beta 26-Jan-2019 Phillip Summers difficultylevelhigh@gmail.com"
Changed lines of the file:
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@@
     (thickness 1.6002)
     (drawings 21)
-    (tracks 4229)
+    (tracks 4218)
     (zones 0)
-    (modules 98)
+    (modules 97)
     (nets 285)
   )
   (page A4)
   (title_block
-    (date 2019-01-26)
+    (date 2019-02-17)
   )
   (layers
@@
       (effects (font (size 1.524 1.524) (thickness 0.3048)))
     )
-    (fp_text value SUPER (at 0 -2.54 90) (layer F.SilkS)
+    (fp_text value 0.22F (at 0 -2.54 90) (layer F.SilkS)
       (effects (font (size 1.524 1.3335) (thickness 0.3048)))
     )
@@
     )
   )
-  (module Connector_PinHeader_2.54mm:PinHeader_1x02_P2.54mm_Vertical (layer Component)
-    (at 88.519 109.474)
-    (descr "Through hole straight pin header, 1x02, 2.54mm pitch, single row")
-    (tags "Through hole pin header THT 1x02 2.54mm single row")
-    (fp_text reference BT1 (at 0 -3.4036) (layer F.SilkS)
-      (effects (font (size 1 1) (thickness 0.15)))
-    )
-    (fp_text value SUPER (at -0.0254 -2.2352 180) (layer F.Fab)
-      (effects (font (size 0.5 0.5) (thickness 0.125)))
-    )
-    (fp_text user %R (at 0 1.27 90) (layer F.Fab)
-      (effects (font (size 1 1) (thickness 0.15)))
-    )
-    (fp_line (start 1.8 -1.8) (end -1.8 -1.8) (layer F.CrtYd) (width 0.05))
-    (fp_line (start 1.8 4.35) (end 1.8 -1.8) (layer F.CrtYd) (width 0.05))
-    (fp_line (start -1.8 4.35) (end 1.8 4.35) (layer F.CrtYd) (width 0.05))
-    (fp_line (start -1.8 -1.8) (end -1.8 4.35) (layer F.CrtYd) (width 0.05))
-    (fp_line (start -1.33 -1.33) (end 0 -1.33) (layer F.SilkS) (width 0.12))
-    (fp_line (start -1.33 0) (end -1.33 -1.33) (layer F.SilkS) (width 0.12))
-    (fp_line (start -1.33 1.27) (end 1.33 1.27) (layer F.SilkS) (width 0.12))
-    (fp_line (start 1.33 1.27) (end 1.33 3.87) (layer F.SilkS) (width 0.12))
-    (fp_line (start -1.33 1.27) (end -1.33 3.87) (layer F.SilkS) (width 0.12))
-    (fp_line (start -1.33 3.87) (end 1.33 3.87) (layer F.SilkS) (width 0.12))
-    (fp_line (start -1.27 -0.635) (end -0.635 -1.27) (layer F.Fab) (width 0.1))
-    (fp_line (start -1.27 3.81) (end -1.27 -0.635) (layer F.Fab) (width 0.1))
-    (fp_line (start 1.27 3.81) (end -1.27 3.81) (layer F.Fab) (width 0.1))
-    (fp_line (start 1.27 -1.27) (end 1.27 3.81) (layer F.Fab) (width 0.1))
-    (fp_line (start -0.635 -1.27) (end 1.27 -1.27) (layer F.Fab) (width 0.1))
-    (pad 2 thru_hole oval (at 0 2.54) (size 1.7 1.7) (drill 1) (layers *.Cu *.Mask)
-      (net 154 GND))
-    (pad 1 thru_hole rect (at 0 0) (size 1.7 1.7) (drill 1) (layers *.Cu *.Mask)
-      (net 152 /VBAT1))
-    (model ${KISYS3DMOD}/Connector_PinHeader_2.54mm.3dshapes/PinHeader_1x02_P2.54mm_Vertical.wrl
-      (at (xyz 0 0 0))
-      (scale (xyz 1 1 1))
-      (rotate (xyz 0 0 0))
-    )
-  )
   (module Resistor_THT:R_Axial_DIN0204_L3.6mm_D1.6mm_P7.62mm_Horizontal (layer Component)
     (at 179.832 63.5)
@@
     )
   )
-  (gr_text "Beta 26-Jan-2019 Phillip Summers difficultylevelhigh@gmail.com" (at 236.1184 114.7826 90) (layer F.SilkS)
+  (gr_text "Beta 17-Feb-2019 Phillip Summers difficultylevelhigh@gmail.com" (at 236.1184 114.7826 90) (layer F.SilkS)
     (effects (font (size 1.016 0.712) (thickness 0.178)))
   )
@@
   (segment (start 179.882811 97.383611) (end 183.300001 100.800801) (width 0.6096) (layer Component) (net 152) (status 20))
   (segment (start 183.300001 100.800801) (end 184.15 101.6508) (width 0.6096) (layer Component) (net 152) (status 30))
-  (segment (start 101.687763 92.540199) (end 106.484799 92.540199) (width 0.6096) (layer Component) (net 152) (status 20))
-  (segment (start 96.526763 97.701199) (end 101.687763 92.540199) (width 0.6096) (layer Component) (net 152))
   (segment (start 106.484799 92.540199) (end 107.2896 93.345) (width 0.6096) (layer Component) (net 152) (status 30))
-  (segment (start 88.684199 97.939959) (end 88.795959 97.828199) (width 0.6096) (layer Component) (net 152))
-  (segment (start 88.922959 97.701199) (end 88.684199 97.939959) (width 0.6096) (layer Component) (net 152))
-  (segment (start 96.526763 97.701199) (end 88.922959 97.701199) (width 0.6096) (layer Component) (net 152))
   (segment (start 128.947702 100.58654) (end 126.402162 98.041) (width 0.6096) (layer Component) (net 152))
   (segment (start 124.33 98.041) (end 121.400199 95.111199) (width 0.6096) (layer Component) (net 152))
@@
   (segment (start 126.402162 98.041) (end 124.33 98.041) (width 0.6096) (layer Component) (net 152))
   (segment (start 109.055799 95.111199) (end 107.2896 93.345) (width 0.6096) (layer Component) (net 152) (status 20))
-  (segment (start 88.684199 97.939959) (end 88.684199 102.47895) (width 0.6096) (layer Component) (net 152))
-  (segment (start 88.684199 102.47895) (end 88.976255 102.771006) (width 0.6096) (layer Component) (net 152))
-  (segment (start 88.519 105.486255) (end 88.976255 105.029) (width 0.6096) (layer Component) (net 152))
-  (segment (start 88.519 109.474) (end 88.519 105.486255) (width 0.6096) (layer Component) (net 152))
-  (segment (start 88.976255 102.771006) (end 88.976255 105.029) (width 0.6096) (layer Component) (net 152))
   (segment (start 185.890001 97.319999) (end 186.69 96.52) (width 0.6096) (layer Copper) (net 152))
   (segment (start 185.331199 97.878801) (end 185.890001 97.319999) (width 0.6096) (layer Copper) (net 152))
@@
   (segment (start 93.306801 120.658801) (end 93.306801 128.101199) (width 0.6096) (layer Copper) (net 154))
   (segment (start 91.948 119.3) (end 93.306801 120.658801) (width 0.6096) (layer Copper) (net 154) (status 10))
-  (segment (start 89.074 112.014) (end 91.948 109.14) (width 0.6096) (layer Component) (net 154) (status 30))
-  (segment (start 88.519 112.014) (end 89.074 112.014) (width 0.6096) (layer Component) (net 154) (status 30))
   (segment (start 87.297686 112.014) (end 88.519 112.014) (width 0.6096) (layer Copper) (net 154) (status 20))
   (segment (start 83.185 107.901314) (end 87.297686 112.014) (width 0.6096) (layer Copper) (net 154))
@@
   (segment (start 195.389566 92.900434) (end 195.389566 90.256182) (width 0.6096) (layer Copper) (net 154))
   (segment (start 191.77 96.52) (end 195.389566 92.900434) (width 0.6096) (layer Copper) (net 154))
+  (segment (start 88.519 112.014) (end 91.948 109.14) (width 0.6096) (layer Component) (net 154) (status 30))
+  (via (at 88.519 112.014) (size 0.889) (drill 0.5842) (layers Component Copper) (net 154))
   (via (at 155.54452 83.63712) (size 0.889) (layers Component Copper) (net 155))
   (segment (start 156.21 91.44) (end 156.21 84.3026) (width 0.6096) (layer Copper) (net 155) (status 10))
@@
   (segment (start 107.162579 76.987421) (end 110.960001 73.189999) (width 0.2032) (layer Copper) (net 165) (status 20))
   (segment (start 110.960001 73.189999) (end 111.76 72.39) (width 0.2032) (layer Copper) (net 165) (status 30))
-  (segment (start 87.9475 116.1415) (end 88.519 116.713) (width 0.2032) (layer Component) (net 165))
-  (segment (start 87.731589 98.679) (end 87.731589 102.460302) (width 0.2032) (layer Component) (net 165))
-  (segment (start 87.731589 102.460302) (end 88.315844 103.044557) (width 0.2032) (layer Component) (net 165))
-  (segment (start 88.315844 104.4575) (end 87.249 105.524344) (width 0.2032) (layer Component) (net 165))
-  (segment (start 87.249 105.524344) (end 87.249 115.443) (width 0.2032) (layer Component) (net 165))
-  (segment (start 88.315844 103.044557) (end 88.315844 104.4575) (width 0.2032) (layer Component) (net 165))
-  (segment (start 87.249 115.443) (end 87.9475 116.1415) (width 0.2032) (layer Component) (net 165))
+  (segment (start 87.731589 102.460302) (end 87.731589 98.679) (width 0.2032) (layer Component) (net 165))
+  (segment (start 88.315844 103.044557) (end 87.731589 102.460302) (width 0.2032) (layer Component) (net 165))
+  (segment (start 88.315844 104.4575) (end 88.315844 103.044557) (width 0.2032) (layer Component) (net 165))
+  (segment (start 87.503 105.270344) (end 88.315844 104.4575) (width 0.2032) (layer Component) (net 165))
+  (segment (start 87.503 115.697) (end 87.503 105.270344) (width 0.2032) (layer Component) (net 165))
+  (segment (start 88.519 116.713) (end 87.503 115.697) (width 0.2032) (layer Component) (net 165))
   (segment (start 121.348499 117.411501) (end 120.65 118.11) (width 0.2032) (layer Component) (net 166) (status 30))
   (segment (start 124.345601 114.414399) (end 121.348499 117.411501) (width 0.2032) (layer Component) (net 166) (status 20))

Commit message: Version Q
Connections:
- net /DTR_TTL renamed Net-(U1-Pad33)
- U1 pad 37: /DSR_TTL -> GND
- U1 pad 38: Net-(U1-Pad38) -> GND
- U1 pad 39: Net-(U1-Pad39) -> VCC
Routing:
- net VCC: track 895.1 -> 935.7 mm
- net /DTR: track 60.3 -> 48.8 mm
- net GND: track 943.9 -> 951.8 mm
- net /D0: track 272.1 -> 275.9 mm
- net /B_A12: track 30.5 -> 32.8 mm
- net /D1: track 295.4 -> 297.5 mm
- net /D2: track 294.5 -> 296.5 mm
- net /PC2: track 116.1 -> 117.5 mm
- net Net-(K10-Pad2): track 122.1 -> 123.3 mm
- net /A14: track 174.2 -> 173.0 mm
- net /RTS_TTL: track 125.3 -> 124.2 mm
- net /TX: track 78.0 -> 77.0 mm
- net /PB1: track 93.8 -> 94.6 mm
- net /PC1: track 100.4 -> 101.1 mm
- net /PC0: track 104.3 -> 105.0 mm
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Other:
- board text added: "Version Q 7-Mar-2019 Phillip Summers difficultylevelhigh@gmail.com"
- board text removed: "Beta 17-Feb-2019 Phillip Summers difficultylevelhigh@gmail.com"
