File: SBC.kicad_pcb (KiCad board)
At the start: 2 copper layers, 160 x 100.3 mm, 97 parts, among them K1 A17, K10 BNKSEL, K11 16K/32K, K12 INTSEL, K13 RSTSEL, K6 A18, K7 128/512, K8 A19, K9 PWR, P1 IDE, P2 POWER, P3 SERIAL, P4 CLK_CPU, P5 CLK_UART, P6 RESET, Q1 2N3906, SW1 RESETSW, U1 16550, U10 74LS243, U11 74LS245, U12 74LS174, U13 74LS174, U14 74LS32, U15 74LS32, U16 74LS32, U17 74LS244, U18 74LS174, U19 8255, U2 27C080, U20 C96ABC, U21 DS1302, U22 MAX232, U23 SRAM_512KO, U24 Z80-CPU, U25 DS1210, U26 74LS06N, U27 74LS14, U3 74LS08, U4 74LS10, U5 74LS125, U6 74LS139, U7 74LS14, U8 74LS245, U9 74LS245, X1 CRYSTAL

Commit message: Version R
Routing:
- net (no net): track 0.00 -> 6.23 mm
Other:
- board text added: "Version R 5-Apr-2019 Phillip Summers difficultylevelhigh@gmail.com"
- board text removed: "Version Q 7-Mar-2019 Phillip Summers difficultylevelhigh@gmail.com"

Commit message: Version S
Parts:
- removed JP1: BATSEL, Connector_PinHeader_2.54mm:PinHeader_1x02_P2.54mm_Vertical
- removed P6: RESET, Connector_PinHeader_2.54mm:PinHeader_1x02_P2.54mm_Vertical
- added G***: LOGO, phil.summers:SOLDERBRIDGES, B.Cu at (150.0, 143.5)
- added G***: LOGO, phil.summers:JUMPERSET3, B.Cu at (144.8, 123.5)
- added G***: LOGO, phil.summers:JUMPERSET2, B.Cu at (144.7, 104.1)
- added G***: LOGO, phil.summers:EPROM JUMPERS, B.Cu at (149.7, 63.6)
- added J1: BATSEL, Connector_PinHeader_2.54mm:PinHeader_2x03_P2.54mm_Vertical, F.Cu at (186.7, 106.7)
- added JP5: RXD, Jumper:SolderJumper-2_P1.3mm_Open_RoundedPad1.0x1.5mm, B.Cu at (113.6, 105.5)
- added JP6: CTS, Jumper:SolderJumper-2_P1.3mm_Open_RoundedPad1.0x1.5mm, B.Cu at (106.0, 105.5)
- added JP7: TXD, Jumper:SolderJumper-2_P1.3mm_Open_RoundedPad1.0x1.5mm, B.Cu at (109.9, 105.5)
- added JP8: RTS, Jumper:SolderJumper-2_P1.3mm_Open_RoundedPad1.0x1.5mm, B.Cu at (102.3, 105.5)
- added P7: BITOUT, Connector_PinHeader_2.54mm:PinHeader_1x02_P2.54mm_Vertical, F.Cu at (117.9, 89.8)
- C28: value 1uF -> 10uF; footprint Capacitor_THT:CP_Radial_Tantal_D4.5mm_P2.50mm -> Capacitor_THT:CP_Radial_D5.0mm_P2.50mm
- moved RR2 32.3 mm to (190.5, 134.5), turned to 180 degrees
- moved K11 12.5 mm to (168.9, 101.6)
- moved C2 12.2 mm to (177.6, 73.7)
- moved D2 10.4 mm to (187.5, 69.3), turned to 180 degrees
- moved SW1 10.1 mm to (181.5, 56.3)
- moved K10 9.16 mm to (168.9, 111.8)
- moved R1 3.05 mm to (179.8, 66.5)
- moved R2 2.90 mm to (187.5, 63.9)
- moved K12 2.64 mm to (190.6, 106.7)
- moved JP4 1.27 mm to (189.4, 92.7)
- moved K8 1.27 mm to (168.9, 132.1)
- moved K6 1.27 mm to (168.9, 121.9)
- moved JP3 1.27 mm to (185.4, 92.7)
- moved U25 1.27 mm to (185.4, 96.5)
Connections:
- net /NC_A23 renamed /~B_IQ0
- C34 pad 1: /VBAT1 -> Net-(C34-Pad1)
- RR2 pad 2: //INT -> /PU1K-A
- RR2 pad 4: /PU1K-A -> //INT
- U21 pad 8: /VBAT1 -> Net-(C34-Pad1)
- U25 pad 7: GND -> /VBAT2
Routing:
- net Net-(C34-Pad1): track 0.00 -> 111.8 mm
- net /VBAT1: track 114.8 -> 6.64 mm
- net //NMI: track 89.3 -> 39.6 mm, vias 1 -> 0
- net /PU1K-C: track 61.2 -> 14.2 mm
- net /PU1K-A: track 50.9 -> 13.8 mm, vias 1 -> 0
- net //INT: track 62.6 -> 35.1 mm, vias 2 -> 0
- net /A14: track 173.0 -> 199.3 mm, vias 2 -> 3
- net /PU1K-B: track 40.3 -> 14.8 mm, vias 1 -> 0
- net /VBAT2: track 0.00 -> 24.5 mm
- net /A15: track 211.9 -> 232.9 mm
- net //CS_ROM: track 70.7 -> 87.6 mm
- net Net-(K11-Pad2): track 39.9 -> 55.2 mm
- net /RTS_TTL: track 124.2 -> 137.7 mm, vias 1 -> 2
- net Net-(P7-Pad1): track 0.00 -> 12.4 mm
- net VCC: track 935.7 -> 926.9 mm
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Other:
- board text added: "SBC VER 2-004s"
- board text added: "Version S 11-Jun-2019 Phillip Summers difficultylevelhigh@gmail.com"
- board text removed: "SBC VER 2-004"
- board text removed: "Version R 5-Apr-2019 Phillip Summers difficultylevelhigh@gmail.com"

Commit message: Version T
Parts:
- removed G***: LOGO, phil.summers:SOLDERBRIDGES
- removed G***: LOGO, phil.summers:JUMPERSET3
- removed G***: LOGO, phil.summers:JUMPERSET2
- removed G***: LOGO, phil.summers:EPROM JUMPERS
- removed J1: BATSEL, Connector_PinHeader_2.54mm:PinHeader_2x03_P2.54mm_Vertical
- added JP1: BATSEL, Connector_PinHeader_2.54mm:PinHeader_1x02_P2.54mm_Vertical, F.Cu at (183.9, 101.6)
- added P6: RESET, Connector_PinHeader_2.54mm:PinHeader_1x02_P2.54mm_Vertical, F.Cu at (182.6, 56.5)
- added U28: 74LS74, Package_DIP:DIP-14_W7.62mm, F.Cu at (178.3, 151.1)
- C28: value 10uF -> 1uF; footprint Capacitor_THT:CP_Radial_D5.0mm_P2.50mm -> Capacitor_THT:CP_Radial_Tantal_D4.5mm_P2.50mm
- moved RR2 32.3 mm to (168.9, 110.5), turned to 90 degrees
- moved C13 31.6 mm to (191.9, 133.3)
- moved P4 17.6 mm to (187.1, 130.6), turned to 270 degrees
- moved C2 12.2 mm to (177.5, 85.9)
- moved K10 11.3 mm to (172.7, 101.1)
- moved D2 10.4 mm to (177.2, 68.5), turned to 270 degrees
- moved SW1 10.1 mm to (180.3, 66.3)
- moved K11 7.74 mm to (176.6, 101.1)
- moved K12 5.57 mm to (188.2, 101.7), turned to 90 degrees
- moved U7 4.93 mm to (177.8, 114.5)
- moved U26 4.22 mm to (177.9, 126.6)
- moved R1 3.05 mm to (179.8, 63.5)
- moved R2 2.90 mm to (187.5, 61.0)
- moved U9 2.54 mm to (198.1, 151.1)
- moved JP4 1.27 mm to (188.1, 92.7)
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Connections:
- net /~B_IQ0 renamed /NC_A23
- net Net-(P7-Pad1) renamed /TURBO
- C34 pad 1: Net-(C34-Pad1) -> /VBAT1
- P4 pad 5: /CLK_CPU -> Net-(P4-Pad5)
- RR2 pad 2: /PU1K-A -> //INT
- RR2 pad 4: //INT -> /PU1K-A
- U21 pad 8: Net-(C34-Pad1) -> /VBAT1
- U25 pad 7: /VBAT2 -> GND
- U26 pad 12: /PU1K-C -> Net-(U26-Pad12)
- U26 pad 13: Net-(U26-Pad13) -> Net-(P4-Pad5)
Routing:
- net Net-(C34-Pad1): track 111.8 -> 0.00 mm
- net /VBAT1: track 6.64 -> 110.0 mm
- net //NMI: track 39.6 -> 94.5 mm, vias 0 -> 1
- net /PU1K-C: track 14.2 -> 52.5 mm
- net //INT: track 35.1 -> 67.4 mm, vias 0 -> 2
- net Net-(U15-Pad6): track 39.3 -> 7.62 mm
- net /PU1K-A: track 13.8 -> 42.9 mm, vias 0 -> 1
- net /A14: track 199.3 -> 172.4 mm, vias 3 -> 2
- net /PU1K-B: track 14.8 -> 41.6 mm, vias 0 -> 1
- net /VBAT2: track 24.5 -> 0.00 mm
- net Net-(P4-Pad5): track 0.00 -> 21.7 mm
- net /A15: track 232.9 -> 211.5 mm
- net Net-(K11-Pad2): track 55.2 -> 37.9 mm
- net GND: track 948.2 -> 932.1 mm
- net //RD: track 282.9 -> 298.0 mm
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Other:
- board text added: "SBC VER 2-004"
- board text added: "Version S 11-May-2019 Phillip Summers difficultylevelhigh@gmail.com"
- board text removed: "SBC VER 2-004s"
- board text removed: "Version S 11-Jun-2019 Phillip Summers difficultylevelhigh@gmail.com"

Commit message: Version U
Parts:
- removed JP1: BATSEL, Connector_PinHeader_2.54mm:PinHeader_1x02_P2.54mm_Vertical
- removed P6: RESET, Connector_PinHeader_2.54mm:PinHeader_1x02_P2.54mm_Vertical
- removed P7: BITOUT, Connector_PinHeader_2.54mm:PinHeader_1x02_P2.54mm_Vertical
- added G***: LOGO, phil.summers:SOLDERBRIDGES, B.Cu at (150.0, 143.5)
- added G***: LOGO, phil.summers:JUMPERSET3, B.Cu at (144.8, 123.5)
- added G***: LOGO, phil.summers:JUMPERSET2, B.Cu at (144.7, 104.1)
- added G***: LOGO, phil.summers:EPROM JUMPERS, B.Cu at (149.7, 63.6)
- added J1: BATSEL, Connector_PinHeader_2.54mm:PinHeader_2x03_P2.54mm_Vertical, F.Cu at (181.2, 95.1)
- C28: value 1uF -> 10uF; footprint Capacitor_THT:CP_Radial_Tantal_D4.5mm_P2.50mm -> Capacitor_THT:CP_Radial_D5.0mm_P2.50mm
- moved U28 43.2 mm to (177.8, 107.9)
- moved RR2 32.3 mm to (190.5, 134.5), turned to 180 degrees
- moved C13 31.6 mm to (223.5, 134.7)
- moved P4 17.6 mm to (181.6, 147.3), turned to 90 degrees
- moved K12 15.2 mm to (173.0, 101.6), turned to 180 degrees
- moved C2 12.2 mm to (177.6, 73.7)
- moved K10 11.3 mm to (168.9, 111.8)
- moved D2 10.4 mm to (187.5, 69.3), turned to 180 degrees
- moved SW1 10.1 mm to (181.5, 56.3)
- moved K11 7.74 mm to (168.9, 101.6)
- moved U7 4.93 mm to (177.8, 119.4)
- moved U26 4.22 mm to (177.8, 130.8)
- moved R1 3.05 mm to (179.8, 66.5)
- moved R2 2.90 mm to (187.5, 63.9)
- moved U9 2.54 mm to (195.6, 151.1)
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Connections:
- net /NC_A23 renamed /~B_IQ0
- net /PU1K-C renamed Net-(RR2-Pad6)
- C34 pad 1: /VBAT1 -> Net-(C34-Pad1)
- RR2 pad 2: //INT -> /PU1K-A
- RR2 pad 4: /PU1K-A -> //INT
- U21 pad 8: /VBAT1 -> Net-(C34-Pad1)
- U25 pad 7: GND -> /VBAT2
Routing:
- net Net-(C34-Pad1): track 0.00 -> 98.5 mm
- net /VBAT1: track 110.0 -> 12.7 mm
- net /TURBO: track 12.4 -> 85.6 mm, vias 0 -> 1
- net /CLK_CPU: track 78.2 -> 147.9 mm, vias 1 -> 5
- net //NMI: track 94.5 -> 39.6 mm, vias 1 -> 0
- net Net-(RR2-Pad6): track 52.5 -> 0.00 mm
- net Net-(P4-Pad5): track 21.7 -> 65.9 mm, vias 0 -> 2
- net /~B_IQ0: track 58.0 -> 101.3 mm
- net GND: track 932.1 -> 966.6 mm, vias 3 -> 4
- net Net-(U15-Pad6): track 7.62 -> 41.1 mm
- net //INT: track 67.4 -> 35.1 mm, vias 2 -> 0
- net /A14: track 172.4 -> 203.9 mm, vias 2 -> 3
- net /PU1K-A: track 42.9 -> 13.8 mm, vias 1 -> 0
- net Net-(U26-Pad12): track 0.00 -> 28.9 mm
- net /PU1K-B: track 41.6 -> 14.8 mm, vias 1 -> 0
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Other:
- board text added: "SBC VER 2-004u"
- board text added: "Version U 14-Jun-2019 Phillip Summers difficultylevelhigh@gmail.com"
- board text removed: "SBC VER 2-004"
- board text removed: "Version S 11-May-2019 Phillip Summers difficultylevelhigh@gmail.com"

Commit message: Version V
Parts:
- removed G***: LOGO, phil.summers:SOLDERBRIDGES
- removed G***: LOGO, phil.summers:JUMPERSET3
- removed G***: LOGO, phil.summers:JUMPERSET2
- removed G***: LOGO, phil.summers:EPROM JUMPERS
- U23: value SRAM_512KO -> AS6C4008-55PCN
Connections:
- net /PU1K-A renamed /PU4K7-A
- net /PU1K-B renamed /PU4K7-B
- net /TURBO renamed /CLKSEL
- P4 pad 5: Net-(P4-Pad5) -> /PU4K7-C
- RR2 pad 6: Net-(RR2-Pad6) -> /PU4K7-C
- U26 pad 13: Net-(P4-Pad5) -> /PU4K7-C
- U28 pad 3: Net-(P4-Pad5) -> /PU4K7-C
Routing:
- net Net-(P4-Pad5): track 65.9 -> 0.00 mm, vias 2 -> 0
- net /PU4K7-C: track 0.00 -> 64.4 mm, vias 0 -> 2
- net /A14: track 203.9 -> 185.8 mm
- net /CLK_CPU: track 147.9 -> 130.8 mm, vias 5 -> 3
- net //CS_RTC: track 168.0 -> 152.4 mm
- net /A10: track 134.6 -> 128.0 mm
- net /CTS: track 49.4 -> 44.4 mm, vias 1 -> 0
- net //IORQ: track 108.1 -> 112.9 mm
- net //NMI: track 39.6 -> 36.6 mm
- net Net-(JP2-Pad2): track 79.6 -> 77.3 mm
- net /B_/HALT: track 195.1 -> 193.4 mm
- net Net-(K11-Pad2): track 53.4 -> 52.0 mm
- net //RD: track 283.5 -> 282.2 mm
- net //IOSEL: track 233.0 -> 231.8 mm
- net //MREQ: track 93.6 -> 94.7 mm
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Other:
- board text added: "*** JUMPER K1 = 1-2, K6 = 1-2, K8 = 1-2"
- board text added: "*** JUMPER K1 = 1-2, K6 = 1-2, K8 = NO JUMPER"
- board text added: "*** JUMPER K1 = 1-2, K6 = 2-3, K8 = 2-3"
- board text added: "128/512"
- board text added: "16K/32K"
- board text added: "1BIT-IN"
- board text added: "A17"
- board text added: "A18"
- board text added: "A19"
- board text added: "BATSEL"
- board text added: "BNKSEL"
- board text added: "BRIDGE IF DS1210 NOT INSTALLED"
- board text added: "BRIDGE IF MAX232 NOT INSTALLED AND"
- board text added: "CTS"
- board text added: "FOR 1Mb 27C080 OR 27C801 EPROM"
- board text added: "FOR 512Kb 27C4001 EPROM"
- board text added: "FOR 512Kb 29F040 OR 49F040 FLASH"
- board text added: "FOR SBC BATTERY BACKUP MODE CONNECT BATTERY GND TO 5 & 6, VCC TO 3"
- board text added: "INTSEL"
- board text added: "JP1"
- board text added: "JP2"
- board text added: "JP2=CLOSED - SWITCH TO VDU CONSOLE IF AVAILABLE"
- board text added: "JP2=OPEN - USE STANDARD SERIAL PORT FOR CONSOLE I/O (DEFAULT)"
- board text added: "JP3"
- board text added: "JP4"
- board text added: "JP5"
- board text added: "JP6"
- board text added: "JP7"
- board text added: "JP8"
- board text added: "K1"
- board text added: "K10"
- board text added: "K10=1-2 RAMTOP IS FIXED (DEFAULT)"
- board text added: "K10=2-3 RAMTOP IS BANKABLE."
- board text added: "K11"
- board text added: "K11=1-2 TOP RAMBANK IS 32Kb (DEFAULT)"
- board text added: "K11=2-3 TOP RAMBANK IS 16Kb"
- board text added: "K12"
- board text added: "K12=1-2 16550 UART INTERRUPT CONNECTED (DEFAULT)"
- board text added: "K12=2-3 16550 UART INTERRUPT DISCONNECTED"
- board text added: "K13"
- board text added: "K13-1-2 N8VEM\LEGACY RESET METHOD"
- board text added: "K13-2-3 KONTRON RESET METHOD (DEFAULT)"
- board text added: "K6"
- board text added: "K6=1-2 IDE PIN 20 CONNECTED TO GND (DEFAULT)"
- board text added: "K6=2-3 IDE PIN 20 CONNECTED TO +5V"
- board text added: "K7"
- board text added: "K7=1-2 FOR AS6C4008 512Kb RAM (DEFAULT)"
- board text added: "K7=2-3 FOR AS6C1008 128Kb RAM"
- board text added: "K8"
- board text added: "K9"
- board text added: "PWR"
- board text added: "RAMCS"
- board text added: "RAMVCC"
- board text added: "ROMWBW CONSOLE SELECT JUMPER"
- board text added: "RSTSEL"
- board text added: "RTC AND RAM BACKED UP BY SUPERCAP JUMPER 3-4, 5-6"
- board text added: "RTC AND RAM BACKUP BY SUPERCAP AND BACKPLANE JUMPER 1-2, 4-6, 3-5"
- board text added: "RTC BACKUP BY SUPERCAP, RAM BACKUP BY BACKPLANE JUMPER 5-6, 1-3 (DEFAULT)"
- board text added: "RTS"
- board text added: "RXD"
- board text added: "SBC VER 2-004v"
- board text added: "TXD"
- board text added: "USING A SERIAL USB-TTL ADAPTER"
- board text added: "Version V 20-Jun-2019 Phillip Summers difficultylevelhigh@gmail.com"
- board text removed: "SBC VER 2-004u"
- board text removed: "Version U 14-Jun-2019 Phillip Summers difficultylevelhigh@gmail.com"

Commit message: Version W
Parts:
- removed K13: RSTSEL, Connector_PinHeader_2.54mm:PinHeader_1x03_P2.54mm_Vertical
- moved R12 20.2 mm to (223.5, 109.2), turned to 270 degrees
Connections:
- RR1 pad 4: /B_/INT -> /B_/BUSRQ
- RR1 pad 5: /B_/NMI -> /B_/INT
- RR1 pad 6: /B_/BUSRQ -> /B_/NMI
- U20 pad C31: /B_/RESET -> Net-(U20-PadC31)
Routing:
- net //RESET_IN: track 117.1 -> 13.4 mm, vias 1 -> 0
- net /B_/RESET: track 55.1 -> 0.00 mm
- net /B_/RESOUT: track 55.7 -> 15.0 mm
- net VCC: track 927.7 -> 941.6 mm
- net /B_/BUSRQ: track 64.3 -> 74.4 mm
- net /B_/HALT: track 193.4 -> 184.8 mm
- net /B_/NMI: track 53.3 -> 61.2 mm
- net /B_A9: track 23.2 -> 17.0 mm
- net /B_/M1: track 77.4 -> 71.4 mm
- net /B_/RFSH: track 32.6 -> 28.6 mm
- net /B_/INT: track 80.2 -> 76.6 mm
- net //BUSAK: track 144.1 -> 147.5 mm, vias 2 -> 1
- net Net-(C34-Pad1): track 98.8 -> 95.5 mm
- net /~B_IQ0: track 101.3 -> 98.1 mm, vias 1 -> 0
- net /B_A11: track 41.5 -> 44.7 mm
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Other:
- board text added: "SBC VER 2-004w"
- board text removed: "K13"
- board text removed: "K13-1-2 N8VEM\LEGACY RESET METHOD"
- board text removed: "K13-2-3 KONTRON RESET METHOD (DEFAULT)"
- board text removed: "RSTSEL"
- board text removed: "SBC VER 2-004v"

Commit message: Version X
Parts:
- moved JP2 10.0 mm to (88.5, 109.2)
- moved R1 9.58 mm to (188.0, 71.6), turned to 90 degrees
- moved D2 5.68 mm to (185.4, 64.0), turned to 270 degrees
- moved R2 4.57 mm to (182.9, 64.0), turned to 270 degrees
- moved C5 1.27 mm to (223.4, 144.8)
Connections:
- U20 pad C31: Net-(U20-PadC31) -> //RESET_IN
Routing:
- net //RESET_IN: track 13.4 -> 153.8 mm
- net /RTS_TTL: track 137.7 -> 86.7 mm, vias 2 -> 3
- net VCC: track 941.6 -> 976.7 mm
- net GND: track 968.2 -> 1002.9 mm, vias 4 -> 3
- net /TX: track 78.8 -> 52.1 mm, vias 2 -> 1
- net /RX: track 71.8 -> 48.4 mm, vias 2 -> 1
- net Net-(JP2-Pad2): track 77.3 -> 66.0 mm
- net /RTS: track 48.4 -> 39.2 mm, vias 1 -> 0
- net /DTR: track 49.0 -> 42.8 mm
- net /A10: track 128.0 -> 133.3 mm
- net /CTS_TTL: track 107.9 -> 102.7 mm
- net /B_/M1: track 71.4 -> 75.7 mm
- net /CTS: track 44.4 -> 47.2 mm
- net /A3: track 186.0 -> 188.8 mm
- net /B_/WAIT: track 83.3 -> 81.5 mm
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Other:
- board text added: "13-Jul-2019 Phillip Summers difficultylevelhigh@gmail.com"
- board text added: "KONTRON ONLY"
- board text added: "SBC VER 2-004x"
- board text removed: "SBC VER 2-004w"
- board text removed: "Version V 20-Jun-2019 Phillip Summers difficultylevelhigh@gmail.com"

Commit message: Version Y
Parts:
- moved R15 0.44 mm to (94.0, 144.0)
- moved LS1 0.29 mm to (80.9, 144.8)
Connections:
- P4 pad 5: /PU4K7-C -> Net-(P4-Pad5)
- U26 pad 12: Net-(U26-Pad12) -> /PU4K7-C
- U26 pad 13: /PU4K7-C -> Net-(P4-Pad5)
- U28 pad 11: Net-(U26-Pad12) -> /PU4K7-C
- U28 pad 3: /PU4K7-C -> Net-(P4-Pad5)
Routing:
- net Net-(P4-Pad5): track 0.00 -> 65.0 mm, vias 0 -> 2
- net VCC: track 976.7 -> 1009.1 mm, vias 2 -> 3
- net Net-(U26-Pad12): track 28.8 -> 0.00 mm
- net /PU4K7-C: track 64.4 -> 43.2 mm, vias 2 -> 0
- net //HALT: track 59.1 -> 71.7 mm
- net /CLK_CPU: track 131.1 -> 139.3 mm
- net /A6: track 145.8 -> 148.0 mm
- net /A4: track 157.1 -> 159.1 mm
- net /D0: track 276.2 -> 274.2 mm
- net Net-(D1-Pad2): track 23.1 -> 22.4 mm
- net /-PC7: track 30.6 -> 30.0 mm
- net /A11: track 159.8 -> 159.2 mm
- net //RESET: track 217.4 -> 216.8 mm
- net Net-(U16-Pad1): track 245.6 -> 245.0 mm
- net GND: track 1002.9 -> 1002.5 mm, vias 3 -> 5
Other:
- board text added: "SBC VER 2-004y"
- board text removed: "SBC VER 2-004x"
