File: SBC.sch (KiCad schematic (older format))
At the start: 93 parts, among them K1 CONN_3, K10 CONN_3, K11 CONN_3, K12 CONN_3, K13 CONN_3, K2 CONN_3, K3 CONN_3, K4 CONN_3, K5 CONN_3, K6 CONN_3, K7 CONN_3, K8 CONN_3, K9 CONN_3, P1 PARALLEL, P2 POWER, P3 SERIAL, P4 CLK_CPU, P5 CLK_UART, P6 RESET, SW1 SW_PUSH, U1 16550, U10 74LS243, U11 74LS245, U12 74LS174, U13 74LS174, U14 74LS32, U15 74LS32, U16 74LS32, U17 74LS244, U18 74LS174, U19 8255, U2 27C080, U20 C96ABC, U21 DS1302, U22 MAX232, U23 SRAM_512KO, U24 Z80-CPU, U25 DS1210, U26 74LS06N, U3 74LS08, U4 74LS10, U5 74LS125, U6 74LS139, U7 74LS14, U8 74LS245, U9 74LS245, X1 CRYSTAL

Commit message: Version B
Parts:
- removed D2: DIODE, D3, symbol SBC-rescue:DIODE
- added D2: 1N4148, Diode_THT:D_DO-35_SOD27_P7.62mm_Horizontal, symbol Diode:1N4148
- added LS1: Speaker, Connector_PinHeader_2.54mm:PinHeader_2x01_P2.54mm_Vertical, symbol Device:Speaker
- added Q1: 2N3906, Package_TO_SOT_THT:TO-92_Inline, symbol Transistor_BJT:2N3906
- added R13, R14: 3K6, Resistor_THT:R_Axial_DIN0204_L3.6mm_D1.6mm_P7.62mm_Horizontal, symbol Device:R
- added R15: 120R, Resistor_THT:R_Axial_DIN0204_L3.6mm_D1.6mm_P7.62mm_Horizontal, symbol Device:R
- BT1, JP1, JP2, P6: footprint SIL-2 -> Connector_PinHeader_2.54mm:PinHeader_1x02_P2.54mm_Vertical
- C1, C10, C11, C12, C13, C14, C15, C16, C17, C18, C19, C20, C21, C22, C23, C29, C3, C30, C32, C4, C5, C6, C7, C8, C9: footprint C2 -> Capacitor_THT:C_Disc_D7.0mm_W2.5mm_P5.00mm
- C2, C31: footprint C1V5 -> Capacitor_THT:CP_Radial_D5.0mm_P2.50mm
- C24, C25, C26, C27, C28: footprint C1V5 -> Capacitor_THT:CP_Radial_Tantal_D4.5mm_P2.50mm
- D1: footprint LEDV -> LED_THT:LED_D5.0mm
- K1, K10, K11, K12, K13, K2, K3, K4, K5, K6, K7, K8, K9: footprint SIL-3 -> Connector_PinHeader_2.54mm:PinHeader_1x03_P2.54mm_Vertical
- P1: footprint pin_array_13x2 -> Connector_PinHeader_2.54mm:PinHeader_2x13_P2.54mm_Vertical
- P2: footprint molex-drive-connector -> (none)
- P3: footprint PIN_ARRAY_5x2 -> Connector_PinHeader_2.54mm:PinHeader_2x05_P2.54mm_Vertical
- P4: footprint 8dip300 -> Package_DIP:DIP-8_W7.62mm_Socket
- P5: footprint 8dip300 -> Oscillator:Oscillator_DIP-8
- R1: value 10 -> 10R; footprint R3 -> Resistor_THT:R_Axial_DIN0204_L3.6mm_D1.6mm_P7.62mm_Horizontal
- R11, R12, R2, R9: footprint R3 -> Resistor_THT:R_Axial_DIN0204_L3.6mm_D1.6mm_P7.62mm_Horizontal
- RR1, RR2: footprint SIL-6 -> Resistor_THT:R_Array_SIP6
- SW1: footprint SW_PUSH_SMALL -> Button_Switch_THT:SW_PUSH_6mm_H8mm
- U1, U19, U24: footprint 40dip600 -> Package_DIP:DIP-40_W15.24mm
- U10, U14, U15, U16, U26, U3, U4, U5, U7: footprint 14dip300 -> Package_DIP:DIP-14_W7.62mm
- U11, U17, U8, U9: footprint 20dip300 -> Package_DIP:DIP-20_W7.62mm
- U12, U13, U18, U22, U6: footprint 16dip300 -> Package_DIP:DIP-16_W7.62mm
- U2: footprint 32dip600 -> Package_DIP:DIP-32_W15.24mm
- U20: footprint C96ABCMC -> (none)
- U21, U25: footprint 8dip300 -> Package_DIP:DIP-8_W7.62mm
- U23: footprint 32dip600 -> Package_DIP:DIP-32_W15.24mm; symbol SRAM_512Ko -> Memory_RAM_Obsolete:SRAM_512Ko
- X1: footprint SIL-2 -> Crystal:Crystal_Round_D3.0mm_Vertical
- hole1, hole2: footprint 1pin -> (none)
Connections:
- wire segments 680 -> 684
- no-connect marks 83 -> 82

Commit message: Version C
Parts:
- JP1: value JUMPER -> BATSEL
- JP2: value JUMPER -> 1BIT-INPUT
- LS1: value Speaker -> SPEAKER
- R12, RR2: value 4700 -> 4K7
- R14: value 3K6 -> 1K8
- R9: value 100 -> 100R
- RR1: value 1000 -> 1K
- SW1: value SW_PUSH -> RESETSW
Connections:
- wire segments 684 -> 685
Other:
- moved on the sheet: R14
Changed lines of the file:
@@
 AR Path="/23C5984C1EADA7" Ref="R12"  Part="1"
 F 0 "R12" V 13930 7400 50  0000 C CNN
-F 1 "4700" V 13850 7400 50  0000 C CNN
+F 1 "4K7" V 13850 7400 50  0000 C CNN
 F 2 "Resistor_THT:R_Axial_DIN0204_L3.6mm_D1.6mm_P7.62mm_Horizontal" V 13950 7400 50  0001 C CNN
 F 3 "" H 13850 7400 50  0001 C CNN
@@
 AR Path="/76BA4C1CDD1C" Ref="RR2"  Part="1"
 F 0 "RR2" V 16500 9650 60  0000 C CNN
-F 1 "4700" V 16600 9650 60  0000 C CNN
+F 1 "4K7" V 16600 9650 60  0000 C CNN
 F 2 "Resistor_THT:R_Array_SIP6" V 16700 9650 60  0001 C CNN
 F 3 "" H 16550 9650 50  0001 C CNN
@@
 AR Path="/76BA4C1694AF" Ref="RR1"  Part="1"
 F 0 "RR1" V 17700 9650 60  0000 C CNN
-F 1 "1000" V 17800 9650 60  0000 C CNN
+F 1 "1K" V 17800 9650 60  0000 C CNN
 F 2 "Resistor_THT:R_Array_SIP6" V 17900 9650 60  0001 C CNN
 F 3 "" H 17750 9650 50  0001 C CNN
@@
 AR Path="/76BA4C0443BA" Ref="SW1"  Part="1"
 F 0 "SW1" H 3700 12660 50  0000 C CNN
-F 1 "SW_PUSH" H 3550 12470 50  0000 C CNN
+F 1 "RESETSW" H 3550 12470 50  0000 C CNN
 F 2 "Button_Switch_THT:SW_PUSH_6mm_H8mm" H 3550 12570 50  0001 C CNN
 F 3 "" H 3550 12550 50  0001 C CNN
@@
 AR Path="/76BA4C02EFF7" Ref="JP2"  Part="1"
 F 0 "JP2" H 1450 11050 60  0000 C CNN
-F 1 "JUMPER" H 1450 10820 40  0000 C CNN
+F 1 "1BIT-INPUT" H 1450 10820 40  0000 C CNN
 F 2 "Connector_PinHeader_2.54mm:PinHeader_1x02_P2.54mm_Vertical" H 1450 10920 40  0001 C CNN
 F 3 "" H 1450 10900 50  0001 C CNN
@@
 AR Path="/76BA4C028868" Ref="JP1"  Part="1"
 F 0 "JP1" H 6200 11000 60  0000 C CNN
-F 1 "JUMPER" H 6200 10770 40  0000 C CNN
+F 1 "BATSEL" H 6200 10770 40  0000 C CNN
 F 2 "Connector_PinHeader_2.54mm:PinHeader_1x02_P2.54mm_Vertical" H 6200 10870 40  0001 C CNN
 F 3 "" H 6200 10850 50  0001 C CNN
@@
 AR Path="/76BA48069BBF" Ref="R9"  Part="1"
 F 0 "R9" V 9430 8000 50  0000 C CNN
-F 1 "100" V 9350 8000 50  0000 C CNN
+F 1 "100R" V 9350 8000 50  0000 C CNN
 F 2 "Resistor_THT:R_Axial_DIN0204_L3.6mm_D1.6mm_P7.62mm_Horizontal" V 9450 8000 50  0001 C CNN
 F 3 "" H 9350 8000 50  0001 C CNN
@@
 L Device:R R14
 U 1 1 5C65AD9D
-P 7000 8000
-F 0 "R14" H 6930 7954 50  0000 R CNN
-F 1 "3K6" H 6930 8045 50  0000 R CNN
-F 2 "Resistor_THT:R_Axial_DIN0204_L3.6mm_D1.6mm_P7.62mm_Horizontal" V 6930 8000 50  0001 C CNN
-F 3 "~" H 7000 8000 50  0001 C CNN
-	1    7000 8000
+P 6750 8000
+F 0 "R14" H 6680 7954 50  0000 R CNN
+F 1 "1K8" H 6680 8045 50  0000 R CNN
+F 2 "Resistor_THT:R_Axial_DIN0204_L3.6mm_D1.6mm_P7.62mm_Horizontal" V 6680 8000 50  0001 C CNN
+F 3 "~" H 6750 8000 50  0001 C CNN
+	1    6750 8000
 	-1   0    0    1
 $EndComp
@@
 P 7200 8850
 F 0 "LS1" H 7370 8846 50  0000 L CNN
-F 1 "Speaker" H 7370 8755 50  0000 L CNN
+F 1 "SPEAKER" H 7370 8755 50  0000 L CNN
 F 2 "Connector_PinHeader_2.54mm:PinHeader_2x01_P2.54mm_Vertical" H 7200 8650 50  0001 C CNN
 F 3 "~" H 7190 8800 50  0001 C CNN
@@
 $EndComp
 Wire Wire Line
-	6750 8350 6750 7850
-Wire Wire Line
 	5900 8350 6400 8350
 $Comp
@@
 Wire Wire Line
 	4850 12200 4850 12400
+Wire Wire Line
+	6750 8150 6750 8350
+Wire Wire Line
+	7000 7850 7000 8150
 $EndSCHEMATC

Commit message: Version D
Parts:
- added unit 3 of U6
- C10, C11, C12, C13, C14, C15, C16, C17, C18, C19, C20, C21, C22, C29, C3, C30, C32, C4, C5, C6, C7, C8, C9: value 0.1 uF -> 0.1uF
- C2: value 10 uF -> 10uF
- C24, C25, C26, C27, C28: value 1.0 uF -> 1uF
- C31: value 22 uF -> 22uF
- JP2: value 1BIT-INPUT -> 1BIT-IN
- K1: value CONN_3 -> A17
- K10: value CONN_3 -> BNKSEL
- K11: value CONN_3 -> 16K/32K
- K12: value CONN_3 -> INTSEL
- K13: value CONN_3 -> RSTSEL
- K2, K4: value CONN_3 -> CTS-DSR
- K3, K5: value CONN_3 -> RTS-DTR
- K6: value CONN_3 -> A18
- K7: value CONN_3 -> 128/512
- K8: value CONN_3 -> A19
- K9: value CONN_3 -> PWR
- U1: symbol SBC-rescue:16550 -> Interface_UART:16550
- U10: symbol SBC-rescue:74LS243 -> 74xx:74LS243
- U11, U8, U9: symbol SBC-rescue:74LS245 -> 74xx:74LS245
- U12, U13, U18: symbol SBC-rescue:74LS174 -> 74xx:74LS174
- U17: symbol SBC-rescue:74LS244 -> 74xx:74LS244
- U19: symbol SBC-rescue:8255 -> Interface:8255
- U2: symbol SBC-rescue:27C080 -> Memory_EPROM:27C080
- U21: symbol SBC-rescue:DS1302 -> Timer_RTC:DS1302+
- U24: symbol SBC-rescue:Z80-CPU -> CPU:Z80CPU
- U6: footprint Package_DIP:DIP-16_W7.62mm -> (none); symbol SBC-rescue:74LS139 -> 74xx:74LS139
Connections:
- wire segments 685 -> 688
- no-connect marks 82 -> 83
Other:
- moved on the sheet: BT1, JP1, LS1, Q1, R13, R14, R15, U17, X1

Commit message: Version E
Parts:
- added JP3: RAMVCC, Jumper:SolderJumper-2_P1.3mm_Open_RoundedPad1.0x1.5mm, symbol Jumper:SolderJumper_2_Open
- added JP4: RAMCS, Jumper:SolderJumper-2_P1.3mm_Open_RoundedPad1.0x1.5mm, symbol Jumper:SolderJumper_2_Open
- added unit 5 of U14
- added unit 5 of U15
- added unit 5 of U16
- added unit 7 of U26
- added unit 5 of U3
- added unit 4 of U4
- added unit 5 of U5
- added unit 7 of U7
- C1, C23: value 0.1 uF -> 0.1uF
- RR1, RR2: symbol SBC-rescue:CONN_6 -> Device:R_Network05
- U14, U15, U16: symbol SBC-rescue:74LS32 -> 74xx:74LS32
- U26: symbol SBC-rescue:74LS06N -> 74xx:74LS06N
- U3: symbol SBC-rescue:74LS08 -> 74xx:74LS08
- U4: symbol SBC-rescue:74LS10 -> 74xx:74LS10
- U5: symbol SBC-rescue:74LS125 -> 74xx:74LS125
- U6: footprint (none) -> Package_DIP:DIP-16_W7.62mm
- U7: symbol SBC-rescue:74LS14 -> 74xx:74LS14
Connections:
- wire segments 688 -> 692
Other:
- moved on the sheet: D1, K10, R9, U26A, U26B, U26C, U26D, U26E, U26F, U6A, U6C, U7A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

Commit message: Version F
Parts:
- removed P6: RESET, Connector_PinHeader_2.54mm:PinHeader_1x02_P2.54mm_Vertical, symbol SBC-rescue:CONN_2
- added JP5: TXRX, Connector_PinHeader_2.54mm:PinHeader_1x02_P2.54mm_Vertical, symbol Connector_Generic:Conn_01x02
- added P6: RESET, Connector_PinHeader_2.54mm:PinHeader_1x02_P2.54mm_Vertical, symbol Connector_Generic:Conn_01x02
- C1, C10, C11, C12, C13, C14, C15, C16, C17, C18, C19, C20, C21, C22, C23, C29, C3, C30, C32, C4, C5, C6, C7, C8, C9: symbol SBC-rescue:C -> Device:C
- C2, C24, C25, C26, C27, C28, C31: symbol SBC-rescue:CP -> Device:CP
- P5: footprint Oscillator:Oscillator_DIP-8 -> Package_DIP:DIP-8_W7.62mm_Socket
Connections:
- wire segments 692 -> 696

Commit message: Version G
Parts:
- removed P1: PARALLEL, Connector_PinHeader_2.54mm:PinHeader_2x13_P2.54mm_Vertical, symbol SBC-rescue:CONN_13X2
- added C33: 0.1uF, Capacitor_THT:C_Disc_D7.0mm_W2.5mm_P5.00mm, symbol Device:C
- added D3: LED, LED_THT:LED_D5.0mm, symbol Device:LED
- added P1: IDE, Connector_PinHeader_2.54mm:PinHeader_2x20_P2.54mm_Vertical, symbol Connector_Generic:Conn_02x20_Odd_Even
- added R16: 470R, Resistor_THT:R_Axial_DIN0204_L3.6mm_D1.6mm_P7.62mm_Horizontal, symbol Device:R
- added U27: 74LS14, Package_DIP:DIP-14_W7.62mm, symbol 74xx:74LS14
- K1, K12, K6, K7, K8, K9: symbol SBC-rescue:CONN_3 -> Connector_Generic:Conn_01x03
Connections:
- net labels added: -PC3, -PC4, -PC5, -PC6, -PC7
- net labels removed: PPWR
- wire segments 696 -> 730
- no-connect marks 83 -> 92
Other:
- moved on the sheet: U19

Commit message: Version I
Parts:
- removed D3: LED, LED_THT:LED_D5.0mm, symbol Device:LED
- removed R16: 470R, Resistor_THT:R_Axial_DIN0204_L3.6mm_D1.6mm_P7.62mm_Horizontal, symbol Device:R
- K10, K11, K13, K2, K3, K4, K5: symbol SBC-rescue:CONN_3 -> Connector_Generic:Conn_01x03
- P1: footprint Connector_PinHeader_2.54mm:PinHeader_2x20_P2.54mm_Vertical -> Connector_IDC:IDC-Header_2x20_P2.54mm_Vertical
- P3: footprint Connector_PinHeader_2.54mm:PinHeader_2x05_P2.54mm_Vertical -> Connector_IDC:IDC-Header_2x05_P2.54mm_Vertical; symbol SBC-rescue:CONN_5X2 -> Connector_Generic:Conn_02x05_Odd_Even
- P4: symbol SBC-rescue:DIL8 -> Oscillator:CXO_DIP8
- P5: footprint Package_DIP:DIP-8_W7.62mm_Socket -> Oscillator:Oscillator_DIP-8; symbol SBC-rescue:DIL8 -> Oscillator:CXO_DIP8
- R1, R11, R12, R2, R9: symbol SBC-rescue:R -> Device:R
- U27: footprint Package_DIP:DIP-14_W7.62mm -> Package_DIP:DIP-14_W7.62mm_Socket
Connections:
- wire segments 730 -> 729
- no-connect marks 92 -> 85
Other:
- moved on the sheet: C1, C2, C23, D1, D2, R1, R11, R12, R2, R9, U7A, U7B

Commit message: Version J
Parts:
- P2: footprint (none) -> Connector_BarrelJack:BarrelJack_CUI_PJ-063AH_Horizontal; symbol SBC-rescue:CONN_4 -> Connector:Barrel_Jack
- U27: footprint Package_DIP:DIP-14_W7.62mm_Socket -> Package_DIP:DIP-14_W7.62mm
Connections:
- wire segments 729 -> 728
- no-connect marks 85 -> 84
Changed lines of the file:
@@
 Sheet 1 1
 Title ""
-Date "2019-01-23"
+Date "2019-01-24"
 Rev ""
 Comp ""
@@
 Wire Wire Line
 	3750 8650 4300 8650
-Connection ~ 2100 12200
-Wire Wire Line
-	2200 12200 2100 12200
 Wire Wire Line
 	4350 12700 4650 12700
@@
 Wire Wire Line
 	2300 12200 2300 12300
-Connection ~ 2300 12200
 Wire Wire Line
 	3750 8550 4300 8550
@@
 Text Label 8250 3100 0    60   ~ 0
 /CS_ROM
-NoConn ~ 2000 12200
 Text Label 8250 13250 0    60   ~ 0
 /CS_CFG1
@@
 $EndComp
 $Comp
-L SBC-rescue:CONN_4 P2
+L Connector:Barrel_Jack P2
 U 1 1 47C1CB92
-P 2150 11850
+P 2200 11900
 AR Path="/773F65F147C1CB92" Ref="P2"  Part="1"
 AR Path="/23C59847C1CB92" Ref="P2"  Part="1"
@@
 AR Path="/5FC47C1CB92" Ref="P2"  Part="1"
 AR Path="/76BA47C1CB92" Ref="P2"  Part="1"
-F 0 "P2" V 2100 11850 50  0000 C CNN
-F 1 "POWER" V 2200 11850 50  0000 C CNN
-F 2 "" V 2300 11850 50  0001 C CNN
-F 3 "" H 2150 11850 50  0001 C CNN
-	1    2150 11850
-	0    -1   -1   0
+F 0 "P2" V 2150 11900 50  0000 C CNN
+F 1 "POWER" V 2250 11900 50  0000 C CNN
+F 2 "Connector_BarrelJack:BarrelJack_CUI_PJ-063AH_Horizontal" V 2350 11900 50  0001 C CNN
+F 3 "" H 2200 11900 50  0001 C CNN
+	1    2200 11900
+	0    1    1    0
 $EndComp
 $Comp
@@
 F 0 "U27" H 3650 5000 50  0000 C CNN
 F 1 "74LS14" H 3650 4900 50  0000 C CNN
-F 2 "Package_DIP:DIP-14_W7.62mm_Socket" H 3650 4650 50  0001 C CNN
+F 2 "Package_DIP:DIP-14_W7.62mm" H 3650 4650 50  0001 C CNN
 F 3 "http://www.ti.com/lit/gpn/sn74LS14" H 3650 4650 50  0001 C CNN
 	1    3650 4650
@@
 F 0 "U27" H 3650 5450 50  0000 C CNN
 F 1 "74LS14" H 3650 5350 50  0000 C CNN
-F 2 "Package_DIP:DIP-14_W7.62mm_Socket" H 3650 5150 50  0001 C CNN
+F 2 "Package_DIP:DIP-14_W7.62mm" H 3650 5150 50  0001 C CNN
 F 3 "http://www.ti.com/lit/gpn/sn74LS14" H 3650 5150 50  0001 C CNN
 	2    3650 5150
@@
 F 0 "U27" H 3650 6017 50  0000 C CNN
 F 1 "74LS14" H 3650 5926 50  0000 C CNN
-F 2 "Package_DIP:DIP-14_W7.62mm_Socket" H 3650 5700 50  0001 C CNN
+F 2 "Package_DIP:DIP-14_W7.62mm" H 3650 5700 50  0001 C CNN
 F 3 "http://www.ti.com/lit/gpn/sn74LS14" H 3650 5700 50  0001 C CNN
 	3    3650 5700
@@
 F 0 "U27" H 3650 6567 50  0000 C CNN
 F 1 "74LS14" H 3650 6476 50  0000 C CNN
-F 2 "Package_DIP:DIP-14_W7.62mm_Socket" H 3650 6250 50  0001 C CNN
+F 2 "Package_DIP:DIP-14_W7.62mm" H 3650 6250 50  0001 C CNN
 F 3 "http://www.ti.com/lit/gpn/sn74LS14" H 3650 6250 50  0001 C CNN
 	4    3650 6250
@@
 F 0 "U27" H 3650 7117 50  0000 C CNN
 F 1 "74LS14" H 3650 7026 50  0000 C CNN
-F 2 "Package_DIP:DIP-14_W7.62mm_Socket" H 3650 6800 50  0001 C CNN
+F 2 "Package_DIP:DIP-14_W7.62mm" H 3650 6800 50  0001 C CNN
 F 3 "http://www.ti.com/lit/gpn/sn74LS14" H 3650 6800 50  0001 C CNN
 	5    3650 6800
@@
 F 0 "U27" H 3650 7667 50  0000 C CNN
 F 1 "74LS14" H 3650 7576 50  0000 C CNN
-F 2 "Package_DIP:DIP-14_W7.62mm_Socket" H 3650 7350 50  0001 C CNN
+F 2 "Package_DIP:DIP-14_W7.62mm" H 3650 7350 50  0001 C CNN
 F 3 "http://www.ti.com/lit/gpn/sn74LS14" H 3650 7350 50  0001 C CNN
 	6    3650 7350
@@
 F 0 "U27" H 19930 2996 50  0000 L CNN
 F 1 "74LS14" H 19930 2905 50  0000 L CNN
-F 2 "Package_DIP:DIP-14_W7.62mm_Socket" H 19700 2950 50  0001 C CNN
+F 2 "Package_DIP:DIP-14_W7.62mm" H 19700 2950 50  0001 C CNN
 F 3 "http://www.ti.com/lit/gpn/sn74LS14" H 19700 2950 50  0001 C CNN
 	7    19700 2950
@@
 Wire Wire Line
 	3200 4650 3350 4650
-Text Label 3200 4650 0    60   ~ 0
+Text Label 3200 6250 0    60   ~ 0
 PC7
 Wire Wire Line
@@
 Wire Wire Line
 	3200 6800 3350 6800
-Text Label 3200 6250 0    60   ~ 0
+Text Label 3200 4650 0    60   ~ 0
 PC4
 NoConn ~ 3200 5150
@@
 Wire Wire Line
 	3950 4650 4100 4650
-Text Label 3950 4650 0    50   ~ 0
+Text Label 3950 6250 0    50   ~ 0
 -PC7
 Wire Wire Line
@@
 Wire Wire Line
 	3950 6800 4100 6800
-Text Label 3950 6250 0    50   ~ 0
+Text Label 3950 4650 0    50   ~ 0
 -PC4
 Text Label 4500 5750 0    50   ~ 0
@@
 Wire Wire Line
 	13500 5500 13500 5700
+Connection ~ 2300 12200
 $EndSCHEMATC
