File: SBC.sch (KiCad schematic (older format))
At the start: 103 parts, among them K1 A17, K10 BNKSEL, K11 16K/32K, K12 INTSEL, K13 RSTSEL, K2 CTS-DSR, K3 RTS-DTR, K4 CTS-DSR, K5 RTS-DTR, K6 A18, K7 128/512, K8 A19, K9 PWR, P1 IDE, P2 POWER, P3 SERIAL, P4 CLK_CPU, P5 CLK_UART, P6 RESET, Q1 2N3906, SW1 RESETSW, U1 16550, U10 74LS243, U11 74LS245, U12 74LS174, U13 74LS174, U14 74LS32, U15 74LS32, U16 74LS32, U17 74LS244, U18 74LS174, U19 8255, U2 27C080, U20 C96ABC, U21 DS1302, U22 MAX232, U23 SRAM_512KO, U24 Z80-CPU, U25 DS1210, U26 74LS06N, U27 74LS14, U3 74LS08, U4 74LS10, U5 74LS125, U6 74LS139, U7 74LS14, U8 74LS245, U9 74LS245, X1 CRYSTAL

Commit message: Version K
Parts:
- D1: value LED -> RUN/HALT
- LS1: value SPEAKER -> SPKR
- P2: footprint Connector_BarrelJack:BarrelJack_CUI_PJ-063AH_Horizontal -> Connector_BarrelJack:BarrelJack_Horizontal
- Q1: footprint Package_TO_SOT_THT:TO-92_Inline -> Package_TO_SOT_THT:TO-92_HandSolder
Changed lines of the file:
@@
 AR Path="/76BA48069BB2" Ref="D1"  Part="1"
 F 0 "D1" H 9900 8100 50  0000 C CNN
-F 1 "LED" H 9900 7900 50  0000 C CNN
+F 1 "RUN/HALT" H 9900 7900 50  0000 C CNN
 F 2 "LED_THT:LED_D5.0mm" H 9900 8000 50  0001 C CNN
 F 3 "" H 9900 8000 50  0001 C CNN
@@
 F 0 "P2" V 2150 11900 50  0000 C CNN
 F 1 "POWER" V 2250 11900 50  0000 C CNN
-F 2 "Connector_BarrelJack:BarrelJack_CUI_PJ-063AH_Horizontal" V 2350 11900 50  0001 C CNN
+F 2 "Connector_BarrelJack:BarrelJack_Horizontal" V 2350 11900 50  0001 C CNN
 F 3 "" H 2200 11900 50  0001 C CNN
 	1    2200 11900
@@
 F 0 "Q1" H 6491 8854 50  0000 L CNN
 F 1 "2N3906" H 6491 8945 50  0000 L CNN
-F 2 "Package_TO_SOT_THT:TO-92_Inline" H 6500 8825 50  0001 L CIN
+F 2 "Package_TO_SOT_THT:TO-92_HandSolder" H 6500 8825 50  0001 L CIN
 F 3 "https://www.fairchildsemi.com/datasheets/2N/2N3906.pdf" H 6300 8900 50  0001 L CNN
 	1    6300 8900
@@
 P 6600 9400
 F 0 "LS1" H 6770 9396 50  0000 L CNN
-F 1 "SPEAKER" H 6770 9305 50  0000 L CNN
+F 1 "SPKR" H 6770 9305 50  0000 L CNN
 F 2 "Connector_PinHeader_2.54mm:PinHeader_2x01_P2.54mm_Vertical" H 6600 9200 50  0001 C CNN
 F 3 "~" H 6590 9350 50  0001 C CNN
@@
 Wire Wire Line
 	3200 5150 3350 5150
-Text Label 3200 6800 0    60   ~ 0
+Text Label 3200 5150 0    60   ~ 0
 PC5
 Wire Wire Line
@@
 Wire Wire Line
 	3200 6250 3350 6250
-Text Label 3200 5700 0    60   ~ 0
+Text Label 3200 4650 0    60   ~ 0
 PC3
 Wire Wire Line
 	3200 6800 3350 6800
-Text Label 3200 4650 0    60   ~ 0
+Text Label 3200 5700 0    60   ~ 0
 PC4
-NoConn ~ 3200 5150
-NoConn ~ 4100 5150
+NoConn ~ 3200 6800
+NoConn ~ 4100 6800
 Wire Wire Line
 	3950 4650 4100 4650
@@
 Wire Wire Line
 	3950 5150 4100 5150
-Text Label 3950 6800 0    50   ~ 0
+Text Label 3950 5150 0    50   ~ 0
 -PC5
 Wire Wire Line
@@
 Wire Wire Line
 	3950 6250 4100 6250
-Text Label 3950 5700 0    50   ~ 0
+Text Label 3950 4650 0    50   ~ 0
 -PC3
 Wire Wire Line
 	3950 6800 4100 6800
-Text Label 3950 4650 0    50   ~ 0
+Text Label 3950 5700 0    50   ~ 0
 -PC4
 Text Label 4500 5750 0    50   ~ 0

Commit message: Version N
Parts:
- removed JP5: TXRX, Connector_PinHeader_2.54mm:PinHeader_1x02_P2.54mm_Vertical, symbol Connector_Generic:Conn_01x02
- removed K2, K4: CTS-DSR, Connector_PinHeader_2.54mm:PinHeader_1x03_P2.54mm_Vertical, symbol Connector_Generic:Conn_01x03
- removed K3, K5: RTS-DTR, Connector_PinHeader_2.54mm:PinHeader_1x03_P2.54mm_Vertical, symbol Connector_Generic:Conn_01x03
- added R16: 470R, Resistor_THT:R_Axial_DIN0204_L3.6mm_D1.6mm_P7.62mm_Horizontal, symbol Device:R
Connections:
- net labels removed: DSR
- wire segments 728 -> 711
- no-connect marks 84 -> 87
Other:
- note removed: "K2 = UART SIDE DSR OR CTS\nK3 = UART SIDE DTR OR RTS\nK4 = SERIAL SIDE DSR OR CTS\nK5 = SERIAL SIDE DTR OR RTS"

Commit message: Version O
Parts:
- added C34: SUPER, library:SuperCap5, symbol SBC-rescue:BATTERY
- BT1: value BATTERY -> SUPER; symbol SBC-rescue:BATTERY -> Connector_Generic:Conn_01x02
Connections:
- wire segments 711 -> 714
Changed lines of the file:
@@
 L SBC-rescue:GND #PWR012
 U 1 1 47EEEA38
-P 6400 10700
+P 6300 10700
 AR Path="/47EEEA38" Ref="#PWR012"  Part="1"
 AR Path="/773F65F147EEEA38" Ref="#PWR012"  Part="1"
@@
 AR Path="/5FC47EEEA38" Ref="#PWR012"  Part="1"
 AR Path="/76BA47EEEA38" Ref="#PWR012"  Part="1"
-F 0 "#PWR012" H 6400 10700 30  0001 C CNN
-F 1 "GND" H 6400 10630 30  0001 C CNN
-F 2 "" H 6400 10700 50  0001 C CNN
-F 3 "" H 6400 10700 50  0001 C CNN
-	1    6400 10700
+F 0 "#PWR012" H 6300 10700 30  0001 C CNN
+F 1 "GND" H 6300 10630 30  0001 C CNN
+F 2 "" H 6300 10700 50  0001 C CNN
+F 3 "" H 6300 10700 50  0001 C CNN
+	1    6300 10700
 	1    0    0    -1
 $EndComp
 $Comp
-L SBC-rescue:BATTERY BT1
+L Connector_Generic:Conn_01x02 BT1
 U 1 1 47EEEA29
-P 6400 10400
+P 6500 10350
 AR Path="/773F65F147EEEA29" Ref="BT1"  Part="1"
 AR Path="/23C59847EEEA29" Ref="BT1"  Part="1"
@@
 AR Path="/5FC47EEEA29" Ref="BT1"  Part="1"
 AR Path="/76BA47EEEA29" Ref="BT1"  Part="1"
-F 0 "BT1" H 6400 10600 50  0000 C CNN
-F 1 "BATTERY" H 6400 10210 50  0000 C CNN
-F 2 "Connector_PinHeader_2.54mm:PinHeader_1x02_P2.54mm_Vertical" H 6400 10310 50  0001 C CNN
-F 3 "" H 6400 10400 50  0001 C CNN
-	1    6400 10400
-	0    1    1    0
+F 0 "BT1" H 6500 10450 50  0000 C CNN
+F 1 "SUPER" H 6500 10160 50  0000 C CNN
+F 2 "Connector_PinHeader_2.54mm:PinHeader_1x02_P2.54mm_Vertical" H 6500 10260 50  0001 C CNN
+F 3 "" H 6500 10350 50  0001 C CNN
+	1    6500 10350
+	1    0    0    -1
 $EndComp
 Text Label 1300 10050 0    60   ~ 0
@@
 Wire Wire Line
 	5550 10700 5950 10700
-Wire Wire Line
-	5950 10100 6400 10100
 Connection ~ 5950 10100
 Wire Wire Line
@@
 $EndComp
 NoConn ~ 13700 4700
+$Comp
+L SBC-rescue:BATTERY BT?
+U 1 1 5C762D3A
+P 6900 10400
+AR Path="/773F65F15C762D3A" Ref="BT?"  Part="1"
+AR Path="/23C5985C762D3A" Ref="BT?"  Part="1"
+AR Path="/DE2D5C762D3A" Ref="BT?"  Part="1"
+AR Path="/25C762D3A" Ref="BT?"  Part="1"
+AR Path="/23BED45C762D3A" Ref="BT?"  Part="1"
+AR Path="/773F8EB45C762D3A" Ref="BT?"  Part="1"
+AR Path="/5C762D3A" Ref="C34"  Part="1"
+AR Path="/95C762D3A" Ref="BT?"  Part="1"
+AR Path="/FFFFFFF05C762D3A" Ref="BT?"  Part="1"
+AR Path="/48EF5C762D3A" Ref="BT?"  Part="1"
+AR Path="/23CC3C5C762D3A" Ref="BT?"  Part="1"
+AR Path="/1290D1E5C762D3A" Ref="BT?"  Part="1"
+AR Path="/23C89C5C762D3A" Ref="BT?"  Part="1"
+AR Path="/26E50145C762D3A" Ref="BT?"  Part="1"
+AR Path="/2600005C762D3A" Ref="BT?"  Part="1"
+AR Path="/23D1A05C762D3A" Ref="BT?"  Part="1"
+AR Path="/5005C762D3A" Ref="BT?"  Part="1"
+AR Path="/23D6C05C762D3A" Ref="BT?"  Part="1"
+AR Path="/23DB0B5C762D3A" Ref="BT?"  Part="1"
+AR Path="/2756B1C5C762D3A" Ref="BT?"  Part="1"
+AR Path="/15C762D3A" Ref="BT?"  Part="1"
+AR Path="/23D8BC5C762D3A" Ref="BT?"  Part="1"
+AR Path="/5FC5C762D3A" Ref="BT?"  Part="1"
+AR Path="/76BA5C762D3A" Ref="BT?"  Part="1"
+F 0 "C34" H 6900 10600 50  0000 C CNN
+F 1 "SUPER" H 6900 10210 50  0000 C CNN
+F 2 "library:SuperCap5" H 6900 10310 50  0001 C CNN
+F 3 "" H 6900 10400 50  0001 C CNN
+	1    6900 10400
+	0    1    1    0
+$EndComp
+$Comp
+L SBC-rescue:GND #PWR0149
+U 1 1 5C7630C6
+P 6900 10700
+AR Path="/5C7630C6" Ref="#PWR0149"  Part="1"
+AR Path="/773F65F15C7630C6" Ref="#PWR?"  Part="1"
+AR Path="/23BED45C7630C6" Ref="#PWR?"  Part="1"
+AR Path="/23C5985C7630C6" Ref="#PWR?"  Part="1"
+AR Path="/773F8EB45C7630C6" Ref="#PWR?"  Part="1"
+AR Path="/25C7630C6" Ref="#PWR?"  Part="1"
+AR Path="/95C7630C6" Ref="#PWR?"  Part="1"
+AR Path="/FFFFFFF05C7630C6" Ref="#PWR?"  Part="1"
+AR Path="/71126E5C7630C6" Ref="#PWR?"  Part="1"
+AR Path="/48EF5C7630C6" Ref="#PWR?"  Part="1"
+AR Path="/23CC3C5C7630C6" Ref="#PWR?"  Part="1"
+AR Path="/1290D1E5C7630C6" Ref="#PWR?"  Part="1"
+AR Path="/6FF0DD405C7630C6" Ref="#PWR?"  Part="1"
+AR Path="/23C89C5C7630C6" Ref="#PWR?"  Part="1"
+AR Path="/26E50145C7630C6" Ref="#PWR?"  Part="1"
+AR Path="/2600005C7630C6" Ref="#PWR?"  Part="1"
+AR Path="/5005C7630C6" Ref="#PWR?"  Part="1"
+AR Path="/2756B1C5C7630C6" Ref="#PWR?"  Part="1"
+AR Path="/15C7630C6" Ref="#PWR?"  Part="1"
+AR Path="/23D8BC5C7630C6" Ref="#PWR?"  Part="1"
+AR Path="/70F26E5C7630C6" Ref="#PWR?"  Part="1"
+AR Path="/23DB0B5C7630C6" Ref="#PWR?"  Part="1"
+AR Path="/5FC5C7630C6" Ref="#PWR?"  Part="1"
+AR Path="/76BA5C7630C6" Ref="#PWR?"  Part="1"
+F 0 "#PWR0149" H 6900 10700 30  0001 C CNN
+F 1 "GND" H 6900 10630 30  0001 C CNN
+F 2 "" H 6900 10700 50  0001 C CNN
+F 3 "" H 6900 10700 50  0001 C CNN
+	1    6900 10700
+	1    0    0    -1
+$EndComp
+Wire Wire Line
+	5950 10100 6300 10100
+Wire Wire Line
+	6300 10350 6300 10100
+Wire Wire Line
+	6300 10450 6300 10700
+Connection ~ 6300 10100
+Wire Wire Line
+	6300 10100 6900 10100
 $EndSCHEMATC

Commit message: Version P
Parts:
- removed BT1: SUPER, Connector_PinHeader_2.54mm:PinHeader_1x02_P2.54mm_Vertical, symbol Connector_Generic:Conn_01x02
- C34: value SUPER -> 0.22F
Connections:
- wire segments 714 -> 711
Changed lines of the file:
@@
 Sheet 1 1
 Title ""
-Date "2019-01-26"
+Date "2019-02-17"
 Rev ""
 Comp ""
@@
 	-1   0    0    1
 $EndComp
-$Comp
-L SBC-rescue:JUMPER JP?
-U 1 1 4C028868
-P 5950 10400
-AR Path="/7E4600384C028868" Ref="JP?"  Part="1"
-AR Path="/26B00314C028868" Ref="JP?"  Part="1"
-AR Path="/773F8EB44C028868" Ref="JP1"  Part="1"
-AR Path="/23CC3C4C028868" Ref="JP1"  Part="1"
-AR Path="/94C028868" Ref="JP1"  Part="1"
-AR Path="/4C028868" Ref="JP1"  Part="1"
-AR Path="/773F65F14C028868" Ref="JP1"  Part="1"
-AR Path="/23C5984C028868" Ref="JP1"  Part="1"
-AR Path="/18434C028868" Ref="JP1"  Part="1"
-AR Path="/24C028868" Ref="JP1"  Part="1"
-AR Path="/23BED44C028868" Ref="JP1"  Part="1"
-AR Path="/14C028868" Ref="JP1"  Part="1"
-AR Path="/FFFFFFF04C028868" Ref="JP1"  Part="1"
-AR Path="/23D8BC4C028868" Ref="JP1"  Part="1"
-AR Path="/5AD72BC24C028868" Ref="JP1"  Part="1"
-AR Path="/23DB0B4C028868" Ref="JP1"  Part="1"
-AR Path="/5FC4C028868" Ref="JP1"  Part="1"
-AR Path="/76BA4C028868" Ref="JP1"  Part="1"
-F 0 "JP1" H 5950 10550 60  0000 C CNN
-F 1 "BATSEL" H 5950 10320 40  0000 C CNN
-F 2 "Connector_PinHeader_2.54mm:PinHeader_1x02_P2.54mm_Vertical" H 5950 10420 40  0001 C CNN
-F 3 "" H 5950 10400 50  0001 C CNN
-	1    5950 10400
-	0    -1   -1   0
-$EndComp
 Text Label 5550 10700 0    60   ~ 0
 B_BAT
@@
 NoConn ~ 20000 8650
 NoConn ~ 20000 9250
-$Comp
-L SBC-rescue:GND #PWR012
-U 1 1 47EEEA38
-P 6300 10700
-AR Path="/47EEEA38" Ref="#PWR012"  Part="1"
-AR Path="/773F65F147EEEA38" Ref="#PWR012"  Part="1"
-AR Path="/23BED447EEEA38" Ref="#PWR013"  Part="1"
-AR Path="/23C59847EEEA38" Ref="#PWR013"  Part="1"
-AR Path="/773F8EB447EEEA38" Ref="#PWR013"  Part="1"
-AR Path="/247EEEA38" Ref="#PWR"  Part="1"
-AR Path="/947EEEA38" Ref="#PWR013"  Part="1"
-AR Path="/FFFFFFF047EEEA38" Ref="#PWR19"  Part="1"
-AR Path="/71126E47EEEA38" Ref="#PWR09"  Part="1"
-AR Path="/48EF47EEEA38" Ref="#PWR09"  Part="1"
-AR Path="/23CC3C47EEEA38" Ref="#PWR18"  Part="1"
-AR Path="/1290D1E47EEEA38" Ref="#PWR09"  Part="1"
-AR Path="/6FF0DD4047EEEA38" Ref="#PWR08"  Part="1"
-AR Path="/23C89C47EEEA38" Ref="#PWR08"  Part="1"
-AR Path="/26E501447EEEA38" Ref="#PWR08"  Part="1"
-AR Path="/26000047EEEA38" Ref="#PWR08"  Part="1"
-AR Path="/50047EEEA38" Ref="#PWR08"  Part="1"
-AR Path="/2756B1C47EEEA38" Ref="#PWR08"  Part="1"
-AR Path="/147EEEA38" Ref="#PWR011"  Part="1"
-AR Path="/23D8BC47EEEA38" Ref="#PWR011"  Part="1"
-AR Path="/70F26E47EEEA38" Ref="#PWR013"  Part="1"
-AR Path="/23DB0B47EEEA38" Ref="#PWR013"  Part="1"
-AR Path="/5FC47EEEA38" Ref="#PWR012"  Part="1"
-AR Path="/76BA47EEEA38" Ref="#PWR012"  Part="1"
-F 0 "#PWR012" H 6300 10700 30  0001 C CNN
-F 1 "GND" H 6300 10630 30  0001 C CNN
-F 2 "" H 6300 10700 50  0001 C CNN
-F 3 "" H 6300 10700 50  0001 C CNN
-	1    6300 10700
-	1    0    0    -1
-$EndComp
-$Comp
-L Connector_Generic:Conn_01x02 BT1
-U 1 1 47EEEA29
-P 6500 10350
-AR Path="/773F65F147EEEA29" Ref="BT1"  Part="1"
-AR Path="/23C59847EEEA29" Ref="BT1"  Part="1"
-AR Path="/DE2D47EEEA29" Ref="BT1"  Part="1"
-AR Path="/247EEEA29" Ref="BT1"  Part="1"
-AR Path="/23BED447EEEA29" Ref="BT1"  Part="1"
-AR Path="/773F8EB447EEEA29" Ref="BT1"  Part="1"
-AR Path="/47EEEA29" Ref="BT1"  Part="1"
-AR Path="/947EEEA29" Ref="BT1"  Part="1"
-AR Path="/FFFFFFF047EEEA29" Ref="BT1"  Part="1"
-AR Path="/48EF47EEEA29" Ref="BT1"  Part="1"
-AR Path="/23CC3C47EEEA29" Ref="BT1"  Part="1"
-AR Path="/1290D1E47EEEA29" Ref="BT1"  Part="1"
-AR Path="/23C89C47EEEA29" Ref="BT1"  Part="1"
-AR Path="/26E501447EEEA29" Ref="BT1"  Part="1"
-AR Path="/26000047EEEA29" Ref="BT1"  Part="1"
-AR Path="/23D1A047EEEA29" Ref="BT1"  Part="1"
-AR Path="/50047EEEA29" Ref="BT1"  Part="1"
-AR Path="/23D6C047EEEA29" Ref="BT1"  Part="1"
-AR Path="/23DB0B47EEEA29" Ref="BT1"  Part="1"
-AR Path="/2756B1C47EEEA29" Ref="BT1"  Part="1"
-AR Path="/147EEEA29" Ref="BT1"  Part="1"
-AR Path="/23D8BC47EEEA29" Ref="BT1"  Part="1"
-AR Path="/5FC47EEEA29" Ref="BT1"  Part="1"
-AR Path="/76BA47EEEA29" Ref="BT1"  Part="1"
-F 0 "BT1" H 6500 10450 50  0000 C CNN
-F 1 "SUPER" H 6500 10160 50  0000 C CNN
-F 2 "Connector_PinHeader_2.54mm:PinHeader_1x02_P2.54mm_Vertical" H 6500 10260 50  0001 C CNN
-F 3 "" H 6500 10350 50  0001 C CNN
-	1    6500 10350
-	1    0    0    -1
-$EndComp
 Text Label 1300 10050 0    60   ~ 0
 BUF_Q7
@@
 Wire Wire Line
 	5550 10700 5950 10700
-Connection ~ 5950 10100
-Wire Wire Line
-	4600 10100 5950 10100
 Wire Notes Line
 	950  11350 7600 11350
@@
 AR Path="/76BA5C762D3A" Ref="BT?"  Part="1"
 F 0 "C34" H 6900 10600 50  0000 C CNN
-F 1 "SUPER" H 6900 10210 50  0000 C CNN
+F 1 "0.22F" H 6900 10210 50  0000 C CNN
 F 2 "library:SuperCap5" H 6900 10310 50  0001 C CNN
 F 3 "" H 6900 10400 50  0001 C CNN
@@
 $EndComp
 Wire Wire Line
-	5950 10100 6300 10100
-Wire Wire Line
-	6300 10350 6300 10100
-Wire Wire Line
-	6300 10450 6300 10700
-Connection ~ 6300 10100
+	4600 10100 5950 10100
+Connection ~ 5950 10100
+$Comp
+L SBC-rescue:JUMPER JP?
+U 1 1 4C028868
+P 5950 10400
+AR Path="/7E4600384C028868" Ref="JP?"  Part="1"
+AR Path="/26B00314C028868" Ref="JP?"  Part="1"
+AR Path="/773F8EB44C028868" Ref="JP1"  Part="1"
+AR Path="/23CC3C4C028868" Ref="JP1"  Part="1"
+AR Path="/94C028868" Ref="JP1"  Part="1"
+AR Path="/4C028868" Ref="JP1"  Part="1"
+AR Path="/773F65F14C028868" Ref="JP1"  Part="1"
+AR Path="/23C5984C028868" Ref="JP1"  Part="1"
+AR Path="/18434C028868" Ref="JP1"  Part="1"
+AR Path="/24C028868" Ref="JP1"  Part="1"
+AR Path="/23BED44C028868" Ref="JP1"  Part="1"
+AR Path="/14C028868" Ref="JP1"  Part="1"
+AR Path="/FFFFFFF04C028868" Ref="JP1"  Part="1"
+AR Path="/23D8BC4C028868" Ref="JP1"  Part="1"
+AR Path="/5AD72BC24C028868" Ref="JP1"  Part="1"
+AR Path="/23DB0B4C028868" Ref="JP1"  Part="1"
+AR Path="/5FC4C028868" Ref="JP1"  Part="1"
+AR Path="/76BA4C028868" Ref="JP1"  Part="1"
+F 0 "JP1" H 5950 10550 60  0000 C CNN
+F 1 "BATSEL" H 5950 10320 40  0000 C CNN
+F 2 "Connector_PinHeader_2.54mm:PinHeader_1x02_P2.54mm_Vertical" H 5950 10420 40  0001 C CNN
+F 3 "" H 5950 10400 50  0001 C CNN
+	1    5950 10400
+	0    -1   -1   0
+$EndComp
 Wire Wire Line
-	6300 10100 6900 10100
+	5950 10100 6900 10100
 $EndSCHEMATC

Commit message: Version Q
Connections:
- net labels removed: DSR_TTL, DTR_TTL
- wire segments 711 -> 715
- no-connect marks 87 -> 84
Changed lines of the file:
@@
 	8950 6450 8450 6450
 Wire Wire Line
-	8950 5750 8450 5750
-Wire Wire Line
-	8950 5250 8450 5250
-Wire Wire Line
 	8100 9300 8100 9400
 Wire Wire Line
@@
 	1    0    0    -1
 $EndComp
-Text Label 8500 5250 0    60   ~ 0
-DSR_TTL
-Text Label 8500 5750 0    60   ~ 0
-DTR_TTL
 Text Label 8500 6550 0    60   ~ 0
 SOUT_TTL
@@
 NoConn ~ 8450 5950
 NoConn ~ 8450 5650
-NoConn ~ 8450 5150
-NoConn ~ 8450 5050
 Text Label 13050 5000 0    60   ~ 0
 DTR
@@
 Text Label 11700 5900 0    50   ~ 0
 RTS
-NoConn ~ 8950 5750
-NoConn ~ 8950 5850
 $Comp
 L Device:R R16
@@
 Wire Wire Line
 	5950 10100 6900 10100
+Wire Wire Line
+	8450 5250 8950 5250
+NoConn ~ 8450 5750
+$Comp
+L power:VCC #PWR?
+U 1 1 5CAD5A4F
+P 9150 5050
+AR Path="/5CAD5A4F" Ref="#PWR?"  Part="1"
+AR Path="/773F65F15CAD5A4F" Ref="#PWR?"  Part="1"
+AR Path="/23BED45CAD5A4F" Ref="#PWR?"  Part="1"
+AR Path="/23C5985CAD5A4F" Ref="#PWR?"  Part="1"
+AR Path="/773F8EB45CAD5A4F" Ref="#PWR?"  Part="1"
+AR Path="/25CAD5A4F" Ref="#PWR?"  Part="1"
+AR Path="/95CAD5A4F" Ref="#PWR?"  Part="1"
+AR Path="/FFFFFFF05CAD5A4F" Ref="#PWR?"  Part="1"
+AR Path="/71126E5CAD5A4F" Ref="#PWR?"  Part="1"
+AR Path="/48EF5CAD5A4F" Ref="#PWR?"  Part="1"
+AR Path="/23CC3C5CAD5A4F" Ref="#PWR?"  Part="1"
+AR Path="/1290D1E5CAD5A4F" Ref="#PWR?"  Part="1"
+AR Path="/6FF0DD405CAD5A4F" Ref="#PWR?"  Part="1"
+AR Path="/23C89C5CAD5A4F" Ref="#PWR?"  Part="1"
+AR Path="/26E50145CAD5A4F" Ref="#PWR?"  Part="1"
+AR Path="/2600005CAD5A4F" Ref="#PWR?"  Part="1"
+AR Path="/5005CAD5A4F" Ref="#PWR?"  Part="1"
+AR Path="/2756B1C5CAD5A4F" Ref="#PWR?"  Part="1"
+AR Path="/15CAD5A4F" Ref="#PWR?"  Part="1"
+AR Path="/23D8BC5CAD5A4F" Ref="#PWR?"  Part="1"
+AR Path="/70F26E5CAD5A4F" Ref="#PWR?"  Part="1"
+AR Path="/23DB0B5CAD5A4F" Ref="#PWR?"  Part="1"
+AR Path="/5FC5CAD5A4F" Ref="#PWR?"  Part="1"
+AR Path="/76BA5CAD5A4F" Ref="#PWR?"  Part="1"
+F 0 "#PWR?" H 9150 5150 30  0001 C CNN
+F 1 "VCC" H 9150 5150 30  0000 C CNN
+F 2 "" H 9150 5050 50  0001 C CNN
+F 3 "" H 9150 5050 50  0001 C CNN
+	1    9150 5050
+	1    0    0    -1
+$EndComp
+Wire Wire Line
+	8450 5150 8950 5150
+Wire Wire Line
+	8950 5150 8950 5250
+$Comp
+L SBC-rescue:GND #PWR?
+U 1 1 5CC9609F
+P 9150 5350
+AR Path="/5CC9609F" Ref="#PWR?"  Part="1"
+AR Path="/773F65F15CC9609F" Ref="#PWR?"  Part="1"
+AR Path="/23BED45CC9609F" Ref="#PWR?"  Part="1"
+AR Path="/23C5985CC9609F" Ref="#PWR?"  Part="1"
+AR Path="/773F8EB45CC9609F" Ref="#PWR?"  Part="1"
+AR Path="/25CC9609F" Ref="#PWR?"  Part="1"
+AR Path="/95CC9609F" Ref="#PWR?"  Part="1"
+AR Path="/FFFFFFF05CC9609F" Ref="#PWR?"  Part="1"
+AR Path="/71126E5CC9609F" Ref="#PWR?"  Part="1"
+AR Path="/48EF5CC9609F" Ref="#PWR?"  Part="1"
+AR Path="/23CC3C5CC9609F" Ref="#PWR?"  Part="1"
+AR Path="/1290D1E5CC9609F" Ref="#PWR?"  Part="1"
+AR Path="/6FF0DD405CC9609F" Ref="#PWR?"  Part="1"
+AR Path="/23C89C5CC9609F" Ref="#PWR?"  Part="1"
+AR Path="/26E50145CC9609F" Ref="#PWR?"  Part="1"
+AR Path="/2600005CC9609F" Ref="#PWR?"  Part="1"
+AR Path="/5005CC9609F" Ref="#PWR?"  Part="1"
+AR Path="/2756B1C5CC9609F" Ref="#PWR?"  Part="1"
+AR Path="/15CC9609F" Ref="#PWR?"  Part="1"
+AR Path="/23D8BC5CC9609F" Ref="#PWR?"  Part="1"
+AR Path="/70F26E5CC9609F" Ref="#PWR?"  Part="1"
+AR Path="/23DB0B5CC9609F" Ref="#PWR?"  Part="1"
+AR Path="/5FC5CC9609F" Ref="#PWR?"  Part="1"
+AR Path="/76BA5CC9609F" Ref="#PWR?"  Part="1"
+F 0 "#PWR?" H 9150 5350 30  0001 C CNN
+F 1 "GND" H 9150 5280 30  0001 C CNN
+F 2 "" H 9150 5350 50  0001 C CNN
+F 3 "" H 9150 5350 50  0001 C CNN
+	1    9150 5350
+	1    0    0    -1
+$EndComp
+Wire Wire Line
+	8950 5250 9150 5250
+Wire Wire Line
+	9150 5250 9150 5350
+Connection ~ 8950 5250
+Wire Wire Line
+	8450 5050 9150 5050
 $EndSCHEMATC

Commit message: Version R
Connections:
- wire segments 715 -> 714
Changed lines of the file:
@@
 EESchema Schematic File Version 4
 LIBS:SBC-cache
-EELAYER 26 0
+EELAYER 29 0
 EELAYER END
 $Descr C 22000 17000
@@
 Sheet 1 1
 Title ""
-Date "2019-02-17"
+Date "2019-04-05"
 Rev ""
 Comp ""
@@
 Text Label 9600 6200 0    60   ~ 0
 SIN_TTL
-Text Label 9600 6000 0    60   ~ 0
-SOUT_TTL
 Text Label 13050 4900 0    60   ~ 0
 TX
@@
 	5300 8550 5950 8550
 Connection ~ 6450 6150
-Wire Wire Line
-	5950 7450 6450 7450
-Connection ~ 6450 7450
-Wire Wire Line
-	6450 7450 6500 7450
 NoConn ~ 8450 6850
 $Comp
@@
 	2300 12700 3250 12700
 Wire Wire Line
-	9550 6000 10050 6000
-Wire Wire Line
 	11650 6000 11950 6000
 $Comp
@@
 	13500 5500 13500 5700
 Connection ~ 2300 12200
-Text Label 9600 6100 0    50   ~ 0
-CTS_TTL
 Text Label 9600 5900 0    50   ~ 0
 RTS_TTL
@@
 Wire Wire Line
 	8450 5050 9150 5050
+Wire Wire Line
+	6450 7450 5950 7450
+Text Label 9600 6100 0    50   ~ 0
+CTS_TTL
+Wire Wire Line
+	9550 6000 10050 6000
+Text Label 9600 6000 0    60   ~ 0
+SOUT_TTL
 $EndSCHEMATC

Commit message: Version S
Parts:
- removed JP1: BATSEL, Connector_PinHeader_2.54mm:PinHeader_1x02_P2.54mm_Vertical, symbol SBC-rescue:JUMPER
- removed P6: RESET, Connector_PinHeader_2.54mm:PinHeader_1x02_P2.54mm_Vertical, symbol Connector_Generic:Conn_01x02
- added J1: BATSEL, Connector_PinHeader_2.54mm:PinHeader_2x03_P2.54mm_Vertical, symbol Connector_Generic:Conn_02x03_Odd_Even
- added JP5: RXD, Jumper:SolderJumper-2_P1.3mm_Open_RoundedPad1.0x1.5mm, symbol Jumper:SolderJumper_2_Open
- added JP6: CTS, Jumper:SolderJumper-2_P1.3mm_Open_RoundedPad1.0x1.5mm, symbol Jumper:SolderJumper_2_Open
- added JP7: TXD, Jumper:SolderJumper-2_P1.3mm_Open_RoundedPad1.0x1.5mm, symbol Jumper:SolderJumper_2_Open
- added JP8: RTS, Jumper:SolderJumper-2_P1.3mm_Open_RoundedPad1.0x1.5mm, symbol Jumper:SolderJumper_2_Open
- added P7: BITOUT, Connector_PinHeader_2.54mm:PinHeader_1x02_P2.54mm_Vertical, symbol Connector_Generic:Conn_01x02
- C28: value 1uF -> 10uF
Connections:
- net labels added: VBAT2, ~B_IQ0
- net labels removed: NC_A23
- wire segments 714 -> 743
- no-connect marks 84 -> 83
Other:
- moved on the sheet: C34, D2, LS1, Q1, R1, R13, R14, R15, R2, SW1
