File: SBC.sch (KiCad schematic (older format))
At the start: 103 parts, among them J1 BATSEL, K1 A17, K10 BNKSEL, K11 16K/32K, K12 INTSEL, K13 RSTSEL, K6 A18, K7 128/512, K8 A19, K9 PWR, P1 IDE, P2 POWER, P3 SERIAL, P4 CLK_CPU, P5 CLK_UART, P7 BITOUT, Q1 2N3906, SW1 RESETSW, U1 16550, U10 74LS243, U11 74LS245, U12 74LS174, U13 74LS174, U14 74LS32, U15 74LS32, U16 74LS32, U17 74LS244, U18 74LS174, U19 8255, U2 27C080, U20 C96ABC, U21 DS1302, U22 MAX232, U23 SRAM_512KO, U24 Z80-CPU, U25 DS1210, U26 74LS06N, U27 74LS14, U3 74LS08, U4 74LS10, U5 74LS125, U6 74LS139, U7 74LS14, U8 74LS245, U9 74LS245, X1 CRYSTAL

Commit message: Version T
Parts:
- removed J1: BATSEL, Connector_PinHeader_2.54mm:PinHeader_2x03_P2.54mm_Vertical, symbol Connector_Generic:Conn_02x03_Odd_Even
- added JP1: BATSEL, Connector_PinHeader_2.54mm:PinHeader_1x02_P2.54mm_Vertical, symbol SBC-rescue:JUMPER
- added P6: RESET, Connector_PinHeader_2.54mm:PinHeader_1x02_P2.54mm_Vertical, symbol Connector_Generic:Conn_01x02
- added U28: 74LS74, Package_DIP:DIP-14_W7.62mm, symbol 74xx:74LS74
- C28: value 10uF -> 1uF
Connections:
- net labels added: NC_A23, TURBO
- net labels removed: VBAT2, ~B_IQ0
- wire segments 743 -> 758
- no-connect marks 83 -> 84
Other:
- moved on the sheet: C1, C34, D2, P4, R1, R2, SW1, U26F

Commit message: Version U
Parts:
- removed JP1: BATSEL, Connector_PinHeader_2.54mm:PinHeader_1x02_P2.54mm_Vertical, symbol SBC-rescue:JUMPER
- removed P6: RESET, Connector_PinHeader_2.54mm:PinHeader_1x02_P2.54mm_Vertical, symbol Connector_Generic:Conn_01x02
- removed P7: BITOUT, Connector_PinHeader_2.54mm:PinHeader_1x02_P2.54mm_Vertical, symbol Connector_Generic:Conn_01x02
- added J1: BATSEL, Connector_PinHeader_2.54mm:PinHeader_2x03_P2.54mm_Vertical, symbol Connector_Generic:Conn_02x03_Odd_Even
- C28: value 1uF -> 10uF; footprint Capacitor_THT:CP_Radial_Tantal_D4.5mm_P2.50mm -> Capacitor_THT:CP_Radial_D5.0mm_P2.50mm
Connections:
- net labels added: VBAT2, ~B_IQ0
- net labels removed: NC_A23, PU1K-C
- wire segments 758 -> 745
Other:
- note removed: "JP1 = ECB BACKPLANE BATTERY (A24)"
- moved on the sheet: C1, C10, C11, C12, C13, C14, C15, C16, C17, C18, C19, C2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

Commit message: Version V
Parts:
- removed U22: MAX232, Package_DIP:DIP-16_W7.62mm, symbol SBC-rescue:MAX232
- removed U23: SRAM_512KO, Package_DIP:DIP-32_W15.24mm, symbol Memory_RAM_Obsolete:SRAM_512Ko
- added U22: MAX232, Package_DIP:DIP-16_W7.62mm, symbol Interface_UART:MAX232
- added U23: AS6C4008-55PCN, Package_DIP:DIP-32_W15.24mm, symbol Memory_RAM:AS6C4008-55PCN
Connections:
- net labels added: CLKSEL, PU4K7-A, PU4K7-B, PU4K7-C
- net labels removed: PU1K-A, PU1K-B, TURBO
- wire segments 745 -> 747
- no-connect marks 84 -> 83
Other:
- moved on the sheet: C23, C24, C25, C26, C27, C28, JP5, JP6, JP7, JP8, K12, K7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

Commit message: Version W
Parts:
- removed K13: RSTSEL, Connector_PinHeader_2.54mm:PinHeader_1x03_P2.54mm_Vertical, symbol Connector_Generic:Conn_01x03
- C34: symbol SBC-rescue:BATTERY -> Device:Battery_Cell
- D1: symbol SBC-rescue:LED -> Device:LED
- JP2: symbol SBC-rescue:JUMPER -> Device:Jumper
- SW1: symbol SBC-rescue:SW_PUSH -> Switch:SW_Push
- U25: symbol SBC-rescue:DS1210 -> Power_Management:DS1210
- X1: symbol SBC-rescue:CRYSTAL -> Device:Crystal
Connections:
- net labels removed: B_/RESET
- wire segments 747 -> 745
- no-connect marks 83 -> 84
Other:
- note added: "SuperCapacitor\n0.22F/0.33F 5V"
- moved on the sheet: C10, C12, C14, C16, C18, C20, C22, C30, C33, C4, C6, C8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

Commit message: Version X
Parts:
- removed hole1, hole2: CONN_1, symbol SBC-rescue:CONN_1
- U20: footprint (none) -> library:C96ABCMC; symbol SBC-rescue:C96ABC -> Connector:C96ABC
Connections:
- wire segments 745 -> 744
Other:
- note removed: "MOUNTING HOLES"
Changed lines of the file:
@@
 	14650 4850 14350 4850
 Wire Wire Line
-	17250 2700 17250 2850
-Connection ~ 17250 2850
-Wire Wire Line
 	16200 6950 15650 6950
 Wire Wire Line
@@
 NoConn ~ 15750 1650
 NoConn ~ 15750 1450
-Text Notes 17050 2600 0    60   ~ 0
-MOUNTING HOLES
-$Comp
-L power:GND #PWR?
-U 1 1 4C016D65
-P 17250 3000
-AR Path="/5AD700384C016D65" Ref="#PWR?"  Part="1"
-AR Path="/2AF00314C016D65" Ref="#PWR?"  Part="1"
-AR Path="/4C016D65" Ref="#PWR07"  Part="1"
-AR Path="/23C89C4C016D65" Ref="#PWR01"  Part="1"
-AR Path="/773F65F14C016D65" Ref="#PWR07"  Part="1"
-AR Path="/23C5984C016D65" Ref="#PWR08"  Part="1"
-AR Path="/B36D4C016D65" Ref="#PWR01"  Part="1"
-AR Path="/23BED44C016D65" Ref="#PWR08"  Part="1"
-AR Path="/71126E4C016D65" Ref="#PWR03"  Part="1"
-AR Path="/6FF0DD404C016D65" Ref="#PWR02"  Part="1"
-AR Path="/26E50144C016D65" Ref="#PWR02"  Part="1"
-AR Path="/94C016D65" Ref="#PWR07"  Part="1"
-AR Path="/2600004C016D65" Ref="#PWR02"  Part="1"
-AR Path="/5004C016D65" Ref="#PWR02"  Part="1"
-AR Path="/2756B1C4C016D65" Ref="#PWR02"  Part="1"
-AR Path="/773F8EB44C016D65" Ref="#PWR08"  Part="1"
-AR Path="/23CC3C4C016D65" Ref="#PWR40"  Part="1"
-AR Path="/FFFFFFF04C016D65" Ref="#PWR39"  Part="1"
-AR Path="/14C016D65" Ref="#PWR05"  Part="1"
-AR Path="/23D8BC4C016D65" Ref="#PWR05"  Part="1"
-AR Path="/70F26E4C016D65" Ref="#PWR07"  Part="1"
-AR Path="/5AD72BC24C016D65" Ref="#PWR05"  Part="1"
-AR Path="/23DB0B4C016D65" Ref="#PWR07"  Part="1"
-AR Path="/5FC4C016D65" Ref="#PWR06"  Part="1"
-AR Path="/76BA4C016D65" Ref="#PWR07"  Part="1"
-F 0 "#PWR07" H 17250 3000 30  0001 C CNN
-F 1 "GND" H 17250 2930 30  0001 C CNN
-F 2 "" H 17250 3000 50  0001 C CNN
-F 3 "" H 17250 3000 50  0001 C CNN
-	1    17250 3000
-	1    0    0    -1
-$EndComp
 Text Label 10200 2250 2    50   ~ 0
 VBAT2
@@
 $EndComp
 $Comp
-L SBC-rescue:CONN_1 P?
-U 1 1 4C002A4E
-P 17400 2850
-AR Path="/384C002A4E" Ref="P?"  Part="1"
-AR Path="/27000314C002A4E" Ref="P?"  Part="1"
-AR Path="/23D7D44C002A4E" Ref="P?"  Part="1"
-AR Path="/23D0B04C002A4E" Ref="hole2"  Part="1"
-AR Path="/23D33B4C002A4E" Ref="hole2"  Part="1"
-AR Path="/773F65F14C002A4E" Ref="hole2"  Part="1"
-AR Path="/23C5984C002A4E" Ref="hole2"  Part="1"
-AR Path="/44C002A4E" Ref="hole2"  Part="1"
-AR Path="/7E44048F4C002A4E" Ref="hole2"  Part="1"
-AR Path="/2FB0D344C002A4E" Ref="hole"  Part="1"
-AR Path="/4C002A4E" Ref="hole2"  Part="1"
-AR Path="/B36D4C002A4E" Ref="hole2"  Part="1"
-AR Path="/24C002A4E" Ref="hole2"  Part="1"
-AR Path="/23BED44C002A4E" Ref="hole2"  Part="1"
-AR Path="/773F8EB44C002A4E" Ref="hole2"  Part="1"
-AR Path="/94C002A4E" Ref="hole2"  Part="1"
-AR Path="/23CC3C4C002A4E" Ref="hole2"  Part="1"
-AR Path="/FFFFFFF04C002A4E" Ref="hole2"  Part="1"
-AR Path="/23C89C4C002A4E" Ref="hole2"  Part="1"
-AR Path="/26E50144C002A4E" Ref="hole2"  Part="1"
-AR Path="/2600004C002A4E" Ref="hole2"  Part="1"
-AR Path="/23D5EB4C002A4E" Ref="hole2"  Part="1"
-AR Path="/5004C002A4E" Ref="hole2"  Part="1"
-AR Path="/23DB0B4C002A4E" Ref="hole2"  Part="1"
-AR Path="/2756B1C4C002A4E" Ref="hole2"  Part="1"
-AR Path="/14C002A4E" Ref="hole2"  Part="1"
-AR Path="/23D8BC4C002A4E" Ref="hole2"  Part="1"
-AR Path="/5AD72BC24C002A4E" Ref="hole2"  Part="1"
-AR Path="/5FC4C002A4E" Ref="hole2"  Part="1"
-AR Path="/76BA4C002A4E" Ref="hole2"  Part="1"
-F 0 "hole2" H 17480 2850 40  0000 L CNN
-F 1 "CONN_1" H 17400 2905 30  0001 C CNN
-F 2 "" H 17400 3005 30  0001 C CNN
-F 3 "" H 17400 2850 50  0001 C CNN
-	1    17400 2850
-	1    0    0    -1
-$EndComp
-$Comp
-L SBC-rescue:CONN_1 P?
-U 1 1 4C002A4A
-P 17400 2700
-AR Path="/7E4600384C002A4A" Ref="P?"  Part="1"
-AR Path="/27000314C002A4A" Ref="P?"  Part="1"
-AR Path="/4C002A4A" Ref="hole1"  Part="1"
-AR Path="/23D0B04C002A4A" Ref="hole1"  Part="1"
-AR Path="/23D33B4C002A4A" Ref="hole1"  Part="1"
-AR Path="/773F65F14C002A4A" Ref="hole1"  Part="1"
-AR Path="/7E44048F4C002A4A" Ref="hole1"  Part="1"
-AR Path="/2330CD04C002A4A" Ref="hole"  Part="1"
-AR Path="/24C002A4A" Ref="hole1"  Part="1"
-AR Path="/23BED44C002A4A" Ref="hole1"  Part="1"
-AR Path="/773F8EB44C002A4A" Ref="hole1"  Part="1"
-AR Path="/23CC3C4C002A4A" Ref="hole1"  Part="1"
-AR Path="/94C002A4A" Ref="hole1"  Part="1"
-AR Path="/23C5984C002A4A" Ref="hole1"  Part="1"
-AR Path="/FFFFFFF04C002A4A" Ref="hole1"  Part="1"
-AR Path="/23C89C4C002A4A" Ref="hole1"  Part="1"
-AR Path="/26E50144C002A4A" Ref="hole1"  Part="1"
-AR Path="/2600004C002A4A" Ref="hole1"  Part="1"
-AR Path="/23D5EB4C002A4A" Ref="hole1"  Part="1"
-AR Path="/5004C002A4A" Ref="hole1"  Part="1"
-AR Path="/23DB0B4C002A4A" Ref="hole1"  Part="1"
-AR Path="/2756B1C4C002A4A" Ref="hole1"  Part="1"
-AR Path="/14C002A4A" Ref="hole1"  Part="1"
-AR Path="/23D8BC4C002A4A" Ref="hole1"  Part="1"
-AR Path="/5AD72BC24C002A4A" Ref="hole1"  Part="1"
-AR Path="/5FC4C002A4A" Ref="hole1"  Part="1"
-AR Path="/76BA4C002A4A" Ref="hole1"  Part="1"
-F 0 "hole1" H 17480 2700 40  0000 L CNN
-F 1 "CONN_1" H 17400 2755 30  0001 C CNN
-F 2 "" H 17400 2855 30  0001 C CNN
-F 3 "" H 17400 2700 50  0001 C CNN
-	1    17400 2700
-	1    0    0    -1
-$EndComp
-$Comp
 L 74xx:74LS125 U5
 U 3 1 4C002905
@@
 CLK_UART
 $Comp
-L SBC-rescue:C96ABC U20
+L Connector:C96ABC U20
 U 1 1 47EAEFC0
-P 20950 10600
+P 20750 10650
 AR Path="/C47EAEFC0" Ref="U20"  Part="1"
 AR Path="/773F65F147EAEFC0" Ref="U20"  Part="1"
@@
 AR Path="/76BA47EAEFC0" Ref="U20"  Part="1"
 AR Path="/3F80000047EAEFC0" Ref="U20"  Part="1"
-F 0 "U20" H 20950 15500 70  0000 C CNN
-F 1 "C96ABC" V 21200 10600 70  0000 C CNN
-F 2 "" V 21300 10600 70  0001 C CNN
-F 3 "" H 20950 10600 50  0001 C CNN
-	1    20950 10600
+F 0 "U20" H 20750 15650 70  0000 C CNN
+F 1 "C96ABC" V 21000 10650 70  0000 C CNN
+F 2 "library:C96ABCMC" V 21100 10650 70  0001 C CNN
+F 3 "" H 20750 10650 50  0001 C CNN
+	1    20750 10650
 	1    0    0    -1
 $EndComp
@@
 	2400 12600 2500 12600
 Wire Wire Line
-	17250 2850 17250 3000
-Wire Wire Line
 	4350 12600 4650 12600
 Wire Wire Line
@@
 	11050 1350 11000 1350
 Connection ~ 11050 1350
-NoConn ~ 20450 15050
+NoConn ~ 20000 15050
 Text Notes 5650 11050 0    50   ~ 0
 SuperCapacitor\n0.22F/0.33F 5V
@@
 Wire Wire Line
 	5950 10450 6500 10450
+Wire Wire Line
+	20000 15050 20450 15050
+Text Label 20000 15050 0    60   ~ 0
+/RESET_IN
 $EndSCHEMATC
